File: controller.kicad_sch (KiCad schematic)
At the start: 48 parts, among them Q1 M_CHG, Q2 M_DSG, Q4 NPN_REGIN, U1 MP2790DFP-0000-T

Commit message: post solar meeting with ezzat
Parts:
- C_PACK_E: MFR (none) -> KEMET; MFR P/N (none) -> A785KN476M1JLAS045; Supplier_1 (none) -> DigiKey; Supplier_1 P/N (none) -> 399-A785KN476M1JLAS045TR-ND; Supplier_1 Price @ QTY (none) -> 0.97; Supplier_1 Unit Price (none) -> 1
Connections:
- net TOP is gone; now on net C6: D_BATT.1 (K), D_CHG_VGS.2 (A), Q1.3 (S), R_CHG_PUP.2, R_PACK_FLT2.2, R_REG.2, R_TOP_FLT.1
- net C5: now also R_CELL_FLT5.1
- net C6: now also R_CELL_FLT6.1
- net GND: now also R_CELL_FLT.1; no longer C_SRN_GND.2, R_SRP_FLT.2, U1.23 (AGND)
- net PGND-E: no longer R_SENSE.2, R_SRN_FLT.1
- net SRN: now also C_SRN_SRP.1, R_SRN_FLT.1; no longer C_SRN_GND.1, C_SRN_SRP.2, R_SRN_FLT.2
- net SRP: now also C_SRN_SRP.2, R_SRP_FLT.2; no longer C_SRN_SRP.1, C_SRP_GND.2, R_SRP_FLT.1
- net BATT+: now reaches C_PACK_E.1, D_DSG_VGS.2 (A), D_PACK_E.1 (K), Q2.3 (S), R_DSG_PUP.2
- new net: C_SRN_GND.2, R_SRN_FLT.2
- new net: C_SRP_GND.2, R_SRP_FLT.1
- new net AGND: U1.23 (AGND)
- new net BATT-: C_SRN_GND.1, R_SENSE.2
Other:
- moved on the sheet: C_3V3, C_CELL_FLT, C_CELL_FLT1, C_CELL_FLT2, C_CELL_FLT3, C_CELL_FLT4, C_CELL_FLT5, C_CP, C_MID, C_PACK_E, C_PACK_FLT2, C_REG1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
