File: input.kicad_sch (KiCad schematic)
At the start: 1 part

Commit message: post solar meeting with ezzat
Parts:
- removed J: Conn_15X4, symbol Connector:Conn_15X4
Changed lines of the file:
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@@
 	(generator_version "9.0")
 	(paper "A4")
-	(symbol
-		(lib_id "Connector:Conn_15X4")
-		(at 72.39 109.22 0)
-		(unit 1)
-		(exclude_from_sim no)
-		(in_bom yes)
-		(on_board yes)
-		(dnp no)
-		(fields_autoplaced yes)
-		(property "Reference" "J"
-			(at 77.47 106.6799 0)
-			(effects
-				(font
-					(size 1.27 1.27)
-				)
-				(justify left)
-			)
-		)
-		(property "Value" "Conn_15X4"
-			(at 77.47 109.2199 0)
-			(effects
-				(font
-					(size 1.27 1.27)
-				)
-				(justify left)
-			)
-		)
-		(property "Footprint" ""
-			(at 72.39 106.68 0)
-			(effects
-				(font
-					(size 1.27 1.27)
-				)
-				(hide yes)
-			)
-		)
-		(property "Datasheet" "~"
-			(at 72.39 106.68 0)
-			(effects
-				(font
-					(size 1.27 1.27)
-				)
-				(hide yes)
-			)
-		)
-		(property "Description" "Connector Europe, 60 contacts, ranges A,B,C,D"
-			(at 72.39 109.22 0)
-			(effects
-				(font
-					(size 1.27 1.27)
-				)
-				(hide yes)
-			)
-		)
-		(pin "C7"
-		)
-		(pin "D3"
-		)
-		(pin "A3"
-		)
-		(pin "A4"
-		)
-		(pin "C3"
-		)
-		(pin "C9"
-		)
-		(pin "A6"
-		)
-		(pin "A15"
-		)
-		(pin "B15"
-		)
-		(pin "D11"
-		)
-		(pin "A12"
-		)
-		(pin "B12"
-		)
-		(pin "C12"
-		)
-		(pin "D12"
-		)
-		(pin "A13"
-		)
-		(pin "B13"
-		)
-		(pin "C13"
-		)
-		(pin "D13"
-		)
-		(pin "A14"
-		)
-		(pin "B14"
-		)
-		(pin "C14"
-		)
-		(pin "D14"
-		)
-		(pin "D6"
-		)
-		(pin "D2"
-		)
-		(pin "A7"
-		)
-		(pin "D9"
-		)
-		(pin "B3"
-		)
-		(pin "D10"
-		)
-		(pin "C10"
-		)
-		(pin "B4"
-		)
-		(pin "B10"
-		)
-		(pin "A11"
-		)
-		(pin "B11"
-		)
-		(pin "C11"
-		)
-		(pin "C15"
-		)
-		(pin "D15"
-		)
-		(pin "B5"
-		)
-		(pin "C8"
-		)
-		(pin "C6"
-		)
-		(pin "D7"
-		)
-		(pin "B8"
-		)
-		(pin "D4"
-		)
-		(pin "D5"
-		)
-		(pin "A10"
-		)
-		(pin "B7"
-		)
-		(pin "C5"
-		)
-		(pin "B6"
-		)
-		(pin "D1"
-		)
-		(pin "B2"
-		)
-		(pin "A2"
-		)
-		(pin "C1"
-		)
-		(pin "B9"
-		)
-		(pin "C2"
-		)
-		(pin "A9"
-		)
-		(pin "A8"
-		)
-		(pin "C4"
-		)
-		(pin "B1"
-		)
-		(pin "D8"
-		)
-		(pin "A1"
-		)
-		(pin "A5"
-		)
-		(instances)
-	)
 )
