File: microcontroller.kicad_sch (KiCad schematic)
At the start: 30 parts, among them J9 Conn_01x02_Socket, U3 RP2350A, X1 ABM8-272-T3

Commit message: Updating stuff
Parts:
- C1, C10, C11, C13, C2, C3, C4, C5, C6, C9: footprint Capacitor_SMD:C_0402_1005Metric -> Capacitor_SMD:C_0603_1608Metric; Mfr Murata Electronics -> YAGEO; Mfr P/N GRM155C71H104JE19D -> CC0603JRX7R9BB104; Supplier_1 P/N 490-GRM155C71H104JE19DTR-ND -> 311-1779-2-ND; Supplier_2 (none) -> JLCPCB; Supplier_2 P/N (none) -> C91183; Supplier_2 Price @ QTY (none) -> 1; Supplier_2 Unit Price (none) -> 0.0042
- C12, C14, C15, C16: footprint Capacitor_SMD:C_0402_1005Metric -> Capacitor_SMD:C_0603_1608Metric; Mfr Murata Electronics -> Murata; Mfr P/N GRM155R60J475ME87D -> GRM188Z71C475KE21D; Supplier_1 Digkey -> Digikey; Supplier_1 P/N 490-5408-2-ND -> 490-GRM188Z71C475KE21DTR-ND; Supplier_1 Unit Price 0.10000 -> 0.25000; Supplier_2 (none) -> JLCPCB; Supplier_2 P/N (none) -> C389010; Supplier_2 Price @ Qty (none) -> 1; Supplier_2 Unit Price (none) -> 0.0710
- C7, C8: footprint Resistor_SMD:R_0201_0603Metric -> Capacitor_SMD:C_0603_1608Metric; Mfr Murata Electronics -> YAGEO; Mfr P/N GRM0335C1E150JA01D -> CC0603FRNPO9BN150; Supplier_1 P/N 490-9658-2-ND -> 311-3887-2-ND; Supplier_1 Unit Price 0.10000 -> 0.14000; Supplier_2 (none) -> JLCPCB; Supplier_2 P/N (none) -> C519483; Supplier_2 Price @ Qty (none) -> 1; Supplier_2 Unit Price (none) -> 0.0098
- R10, R11: footprint Resistor_SMD:R_0201_0603Metric -> Resistor_SMD:R_0603_1608Metric; Mfr P/N RC0201FR-0727RL -> RT0603BRD0727RL; Supplier_1 P/N YAG2554TR-ND -> 13-RT0603BRD0727RLTR-ND; Supplier_1 Unit Price 0.10000 -> 0.14000
- R12: footprint Resistor_SMD:R_0402_1005Metric -> Resistor_SMD:R_0603_1608Metric; Mfr Vishay Dale -> KOA Speer Electronics, Inc.; Mfr P/N TNPW040233R0DEED -> RK73H1JTTD33R0F; Supplier_1 P/N 541-TNPW040233R0DEEDTR-ND -> 2019-RK73H1JTTD33R0FTR-ND; Supplier_1 Unit Price 0.20000 -> 0.10000; Supplier_2 (none) -> JLCPCB; Supplier_2 P/N (none) -> C160041; Supplier_2 Price @ Qty (none) -> 1; Supplier_2 Unit Price (none) -> 0.0041
- R3, R4: footprint Resistor_SMD:R_0201_0603Metric -> Resistor_SMD:R_0603_1608Metric; Mfr P/N AC0201FR-07100RL -> RT0603BRD07100RL; Supplier_1 P/N YAG3412TR-ND -> YAG1497TR-ND; Supplier_1 Unit Price 0.10000 -> 0.14000; Supplier_2 (none) -> JLCPCB; Supplier_2 P/N (none) -> C122970; Supplier_2 Price @ Qty (none) -> 1; Supplier_2 Unit Price (none) -> 0.0214
- R5, R6: footprint Resistor_SMD:R_0402_1005Metric -> Resistor_SMD:R_0603_1608Metric; Mfr KOA Speer Electronics, Inc. -> YAGEO; Mfr P/N RN73R1ETTP3302B25 -> RC0603FR-0733KL; Supplier_1 P/N 2019-RN73R1ETTP3302B25TR-ND -> 311-33.0KHRTR-ND; Supplier_2 (none) -> JLCPCB; Supplier_2 P/N (none) -> C126359; Supplier_2 Price @ Qty (none) -> 1; Supplier_2 Unit Price (none) -> 0.0015
- R7, R9: footprint Resistor_SMD:R_0402_1005Metric -> Resistor_SMD:R_0603_1608Metric; Mfr KOA Speer Electronics, Inc. -> YAGEO; Mfr P/N RK73H1ERTTP1001F -> AC0603FR-071KL; Supplier_1 P/N 2019-RK73H1ERTTP1001FTR-ND -> 311-1KLDTR-ND; Supplier_1 Unit Price 0.13000 -> 0.10000; Supplier_2 (none) -> JLCPCB; Supplier_2 P/N (none) -> C116692; Supplier_2 Price @ Qty (none) -> 1; Supplier_2 Unit Price (none) -> 0.0025
- R8: footprint Resistor_SMD:R_0201_0603Metric -> Resistor_SMD:R_0603_1608Metric; Mfr Bourns Inc. -> YAGEO; Mfr P/N CR0201AFW-1001GAS -> AC0603FR-071KL; Supplier_1 P/N CR0201AFW-1001GASTR-ND -> 311-1KLDTR-ND; Supplier_1 Unit Price 0.1 -> 0.10000; Supplier_2 (none) -> JLCPCB; Supplier_2 P/N (none) -> C116692; Supplier_2 Price @ Qty (none) -> 1; Supplier_2 Unit Price (none) -> 0.0025
Connections:
- net +3V3: now also C16.1; no longer C16.2
- net D-: now also R11.2; no longer R11.1
- net GND: now also C16.2, C8.1; no longer C16.1, C8.2
- net USB_D-: now also R11.1; no longer R11.2
- net XR: now also C8.2; no longer C8.1
- net NSHDN renamed nSHDN
Other:
- moved on the sheet: R3, R5
