File: microcontroller.kicad_sch (KiCad schematic)
At the start: 41 parts, among them U2 W25Q64JVSSIQ, U3 RP2350A, X1 ABM8-272-T3

Commit message: Fixes
Parts:
- C12: Mfr (none) -> YAGEO; Mfr P/N (none) -> CC0201KRX7R5BB104; Supplier_2 (none) -> JLCPCB; Supplier_2 P/N (none) -> C1882920; Supplier_2 Unit Price 0.0042 -> (none)
Changed lines of the file:
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@@
 			)
 		)
-		(property "Description" ""
+		(property "Description" "100nF 6.3V X7R ±10% 0201"
 			(at 259.08 91.44 0)
 			(effects
@@
 			)
 		)
-		(property "Mfr" ""
+		(property "Mfr" "YAGEO"
 			(at 259.08 91.44 0)
 			(effects
@@
 			)
 		)
-		(property "Mfr P/N" ""
+		(property "Mfr P/N" "CC0201KRX7R5BB104"
 			(at 259.08 91.44 0)
 			(effects
@@
 			)
 		)
-		(property "Supplier_2" ""
+		(property "Supplier_2" "JLCPCB"
 			(at 259.08 91.44 0)
 			(effects
@@
 			)
 		)
-		(property "Supplier_2 P/N" ""
+		(property "Supplier_2 P/N" "C1882920"
 			(at 259.08 91.44 0)
 			(effects
@@
 			)
 		)
-		(property "Supplier_2 Unit Price" "0.0042"
+		(property "Supplier_2 Unit Price" ""
 			(at 259.08 91.44 0)
 			(effects
