File: BMS.kicad_pcb (KiCad board)
At the start: 6 copper layers, 44 x 69 mm, 143 parts, among them J1 UJ20-C-H-G-SMT-1-P16-TR, J2 Conn_01x04_Socket, J3 Conn_01x02_Socket, J4 Conn_01x02_Socket, J5 Conn_01x07_Socket, J6 Conn_01x03_Pin, J7 Conn_01x10_Pin, J8 Conn_01x02_Pin, J9 Conn_01x02_Socket, Q1 FZT853TA, Q2 PSMN020-100YS, Q3 PSMN020-100YS, Q4 PSMN3R7-100BSE, Q5 PSMN3R7-100BSE, U1 USBLC6-2SC6, U10 SQ1464EEH-T1_GE3, U11 MP2790DFP-0000-T, U2 USBLC6-2SC6, U3 RP2350A, U4 TPS7B8133QDGNRQ1, U5 SQ1464EEH-T1_GE3, U6 SQ1464EEH-T1_GE3, U7 SQ1464EEH-T1_GE3, U8 SQ1464EEH-T1_GE3, U9 SQ1464EEH-T1_GE3, X1 ABM8-272-T3

Commit message: Updating stuff
Parts:
- removed C_MID1: 100 nF, Capacitor_SMD:C_0402_1005Metric
- added C24: 100 nF, Capacitor_SMD:C_0402_1005Metric, F.Cu at (3.85, 0.48)
- added R17: 10k, Resistor_SMD:R_0603_1608Metric, F.Cu at (182.1, 106.6)
- C1, C10, C11, C13, C2, C3, C4, C5, C6, C9: value 100n -> 100 nF; footprint Capacitor_SMD:C_0201_0603Metric -> Capacitor_SMD:C_0402_1005Metric; moved to F.Cu
- C_PACK_FLT1: moved to F.Cu
- J5: footprint Connector_PinHeader_1.00mm:PinHeader_1x07_P1.00mm_Vertical -> Connector_PinHeader_2.54mm:PinHeader_1x07_P2.54mm_Vertical
- Q1: footprint Package_TO_SOT_SMD:SOT-223-3_TabPin2 -> _BMS:SOT230P700X185-4N
- moved C_PACK_FLT1 184.1 mm to (3.85, 2.46), turned to 0 degrees
- moved R_GATE2 183.7 mm to (0.95, 0.49), turned to 0 degrees
- moved R_GATE3 179.6 mm to (0.95, 2.48), turned to 0 degrees
- moved R_GATE4 175.8 mm to (0.95, 4.47), turned to 0 degrees
- moved R_GATE5 172.2 mm to (0.95, 6.46), turned to 0 degrees
- moved C1 162.2 mm to (8.71, 0.48), turned to 0 degrees
- moved C4 162.2 mm to (8.71, 6.39), turned to 0 degrees
- moved C2 162.0 mm to (8.71, 2.46), turned to 0 degrees
- moved C5 156.6 mm to (8.71, 8.37)
- moved C6 154.9 mm to (11.6, 0.48)
- moved C9 154.3 mm to (11.6, 2.46)
- moved C10 150.9 mm to (11.6, 4.42), turned to 0 degrees
- moved C13 149.2 mm to (11.6, 8.37), turned to 0 degrees
- moved C11 147.5 mm to (11.6, 6.39), turned to 0 degrees
- moved J9 95.0 mm to (81.5, 55.0)
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- renumbered C6 to TP1, C5 to TP2, C4 to TP3, C3 to TP4, C2 to TP5, C1 to TP6, C0 to TP7
Connections:
- C1 pad 1: GND -> +3V3
- C1 pad 2: +3V3 -> GND
- C10 pad 1: +1V1 -> GND
- C10 pad 2: GND -> +1V1
- C11 pad 1: +3V3 -> GND
- C11 pad 2: GND -> +3V3
- C13 pad 1: +3V3 -> GND
- C13 pad 2: GND -> +3V3
- C2 pad 1: GND -> +1V1
- C2 pad 2: +1V1 -> GND
- C3 pad 1: GND -> +3V3
- C3 pad 2: +3V3 -> GND
- C4 pad 1: GND -> +3V3
- C4 pad 2: +3V3 -> GND
- C5 pad 1: GND -> +1V1
- C5 pad 2: +1V1 -> GND
- C6 pad 1: GND -> +3V3
- C6 pad 2: +3V3 -> GND
- C9 pad 1: +3V3 -> GND
- C9 pad 2: GND -> +3V3
- C_PACK_FLT1 pad 1: Net-(U11-PACKP) -> GND
- C_PACK_FLT1 pad 2: GND -> Net-(U11-PACKP)
- U11 pad 30: /main/BMS/NSHDN -> /main/BMS/nSHDN
- U3 pad 15: /main/BMS/NSHDN -> /main/microcontroller/nSHDN
Routing:
- net Net-(Q1-B): track 35.5 -> 0.00 mm, vias 2 -> 0

Commit message: Placement
Parts:
- removed C24, C_SRN_SRP1: 100 nF, Capacitor_SMD:C_0402_1005Metric
- removed G***: LOGO, LOGO
- added C_MID1: 100 nF, Capacitor_SMD:C_0603_1608Metric, F.Cu at (-111.2, 98.0)
- added C_PACK_E2: ~, Capacitor_SMD:C_1206_3216Metric, F.Cu at (279.8, -45.7)
- added C_PACK_E3: ~, Capacitor_SMD:C_1206_3216Metric, F.Cu at (279.8, -42.4)
- added C_SRP_SRN1: 100 nF, Capacitor_SMD:C_0603_1608Metric, F.Cu at (-112.1, 113.7)
- added J10: Conn_01x02_Pin, Connector_JST:JST_PH_S2B-PH-SM4-TB_1x02-1MP_P2.00mm_Horizontal, F.Cu at (36.9, -67.0)
- added J11: Conn_01x02_Pin, Connector_JST:JST_PH_S2B-PH-SM4-TB_1x02-1MP_P2.00mm_Horizontal, F.Cu at (47.1, -67.0)
- added J12: Conn_01x02_Pin, Connector_JST:JST_PH_S2B-PH-SM4-TB_1x02-1MP_P2.00mm_Horizontal, F.Cu at (57.4, -67.0)
- added J13: Conn_01x02_Pin, Connector_JST:JST_PH_S2B-PH-SM4-TB_1x02-1MP_P2.00mm_Horizontal, F.Cu at (67.7, -67.0)
- added R18: 10k, Resistor_SMD:R_0603_1608Metric, F.Cu at (-111.8, 117.7)
- added R19: 10k, Resistor_SMD:R_0603_1608Metric, F.Cu at (-117.0, 117.7)
- added R20: 10k, Resistor_SMD:R_0603_1608Metric, F.Cu at (-109.8, 117.7)
- added R21: 10k, Resistor_SMD:R_0603_1608Metric, F.Cu at (-104.6, 117.7)
- added TP10: CELL0, _BMS:Harwin TP, F.Cu at (-29.8, 103.1)
- added TP8: CELL2, _BMS:Harwin TP, F.Cu at (-29.4, 88.7)
- added TP9: CELL1, _BMS:Harwin TP, F.Cu at (-29.7, 95.8)
- C1, C10, C11, C13, C2, C3, C4, C5, C6, C9, C_CELL_FLT1, C_CELL_FLT2, C_CELL_FLT3, C_CELL_FLT4, C_CELL_FLT5, C_CELL_FLT6, C_PACK_FLT1: footprint Capacitor_SMD:C_0402_1005Metric -> Capacitor_SMD:C_0603_1608Metric
- C12, C14, C15, C16, C19, C20, C21, C22, C23, C_CP1, C_SRN_GND1, C_SRP_GND1: footprint Capacitor_SMD:C_0402_1005Metric -> Capacitor_SMD:C_0603_1608Metric; moved to F.Cu
- C17, C18, C_3V3_1, C_REG1, C_REGIN1, C_TOP_FLT1, C_VDD1, C_VREF1, D1, D11, D2, D3, DAGND_CO1, J1, J3, L1, Q1, R1, R2, R_CHG_PUP1, R_DSG_PUP1, R_REG1, R_SENSE1, R_TOP_FLT1, U1, U11, U2, U3, U4, X1: moved to F.Cu
- C7, C8: footprint Resistor_SMD:R_0201_0603Metric -> Capacitor_SMD:C_0603_1608Metric; moved to F.Cu
- C_PACK_E1: value 47 μF -> ~; moved to F.Cu
- J2: value Conn_01x04_Socket -> Conn_01x02_Socket; footprint Connector_JST:JST_GH_SM04B-GHS-TB_1x04-1MP_P1.25mm_Horizontal -> Connector_AMASS:AMASS_XT30PW-F_1x02_P2.50mm_Horizontal; moved to F.Cu
- J4: value Conn_01x02_Socket -> Conn_01x04_Socket; footprint Connector_AMASS:AMASS_XT30PW-F_1x02_P2.50mm_Horizontal -> Connector_JST:JST_GH_SM04B-GHS-TB_1x04-1MP_P1.25mm_Horizontal
- J5: value Conn_01x07_Socket -> Conn_01x03_Socket; footprint Connector_PinHeader_2.54mm:PinHeader_1x07_P2.54mm_Vertical -> Connector_PinHeader_2.54mm:PinHeader_1x03_P2.54mm_Vertical; moved to F.Cu
- J6: value Conn_01x03_Pin -> Conn_01x03_Socket; footprint Connector_JST:JST_SH_SM03B-SRSS-TB_1x03-1MP_P1.00mm_Horizontal -> Connector_PinHeader_2.54mm:PinHeader_1x03_P2.54mm_Vertical; moved to F.Cu
- J7: value Conn_01x10_Pin -> Conn_01x03_Socket; footprint _BMS:TB4-Hirose -> Connector_PinHeader_2.54mm:PinHeader_1x03_P2.54mm_Vertical
- J8: value Conn_01x02_Pin -> Conn_01x10_Pin; footprint Connector_AMASS:AMASS_XT30PW-M_1x02_P2.50mm_Horizontal -> _BMS:TB4-Hirose
- J9: value Conn_01x02_Socket -> Conn_01x02_Pin; footprint Connector_JST:JST_PH_B2B-PH-K_1x02_P2.00mm_Vertical -> Connector_AMASS:AMASS_XT30PW-M_1x02_P2.50mm_Horizontal
- Q2, Q3: value PSMN020-100YS -> PSMN3R7-100BSE; footprint _BMS:LFPAK56_1 -> _BMS:TO-263-2
- R10: value 27 -> 1k; footprint Resistor_SMD:R_0201_0603Metric -> Resistor_SMD:R_0603_1608Metric; moved to F.Cu
- R11, R8: footprint Resistor_SMD:R_0201_0603Metric -> Resistor_SMD:R_0603_1608Metric; moved to F.Cu
- R12: value 33 -> 27; footprint Resistor_SMD:R_0402_1005Metric -> Resistor_SMD:R_0603_1608Metric; moved to F.Cu
- R13: value 10k -> 33; footprint Resistor_SMD:R_0402_1005Metric -> Resistor_SMD:R_0603_1608Metric; moved to F.Cu
- R14, R15, R16, R5, R9: footprint Resistor_SMD:R_0402_1005Metric -> Resistor_SMD:R_0603_1608Metric; moved to F.Cu
- R3: value 100 -> 1k; footprint Resistor_SMD:R_0201_0603Metric -> Resistor_SMD:R_0603_1608Metric; moved to F.Cu
- R4: value 100 -> 33k; footprint Resistor_SMD:R_0201_0603Metric -> Resistor_SMD:R_0603_1608Metric; moved to F.Cu
- R6: value 33k -> 100; footprint Resistor_SMD:R_0402_1005Metric -> Resistor_SMD:R_0603_1608Metric; moved to F.Cu
- R7: value 1k -> 100; footprint Resistor_SMD:R_0402_1005Metric -> Resistor_SMD:R_0603_1608Metric; moved to F.Cu
- R_CELL_FLT1, R_CELL_FLT2, R_CELL_FLT3, R_CELL_FLT4, R_CELL_FLT5, R_CELL_FLT6, R_CELL_FLT7: value 1000 Ω -> 1k; footprint Resistor_SMD:R_0402_1005Metric -> Resistor_SMD:R_0603_1608Metric
- R_CHG_DRIVER1, R_CHG_MG1, R_CHG_MG2, R_DSG_DRIVER1, R_DSG_MG1, R_DSG_MG2: value 100 Ω -> 100; footprint Resistor_SMD:R_0402_1005Metric -> Resistor_SMD:R_0603_1608Metric
- R_GATE1, R_GATE2, R_GATE3, R_GATE4, R_GATE5, R_GATE6: footprint Resistor_SMD:R_0402_1005Metric -> Resistor_SMD:R_0603_1608Metric
- R_MID1, R_PACK_FLT1: value 100 Ω -> 100; moved to F.Cu
- R_SRN_FLT1, R_SRP_FLT1: value 100 Ω -> 100; footprint Resistor_SMD:R_0402_1005Metric -> Resistor_SMD:R_0603_1608Metric; moved to F.Cu
- TP1: value CELL6 -> TestPoint; footprint _BMS:Harwin TP -> TestPoint:TestPoint_Keystone_5015_Micro_Mini
- TP2: value CELL5 -> TestPoint; footprint _BMS:Harwin TP -> TestPoint:TestPoint_Keystone_5015_Micro_Mini
- TP3: value CELL4 -> TestPoint; footprint _BMS:Harwin TP -> TestPoint:TestPoint_Keystone_5015_Micro_Mini
- TP4: value CELL3 -> CELL6
- TP5: value CELL2 -> CELL5
- TP6: value CELL1 -> CELL4
- TP7: value CELL0 -> CELL3
- moved R_CHG_DRIVER1 305.3 mm to (-131.6, 40.5)
- moved R17 288.9 mm to (-106.6, 117.7), turned to 90 degrees
- moved C_TOP_FLT1 283.7 mm to (-114.4, 98.0), turned to 90 degrees
- moved R_TOP_FLT1 283.7 mm to (-116.0, 98.0), turned to -90 degrees
- moved C_CP1 282.3 mm to (-112.8, 98.0), turned to -90 degrees
- moved R_CHG_PUP1 282.0 mm to (-131.6, 41.8), turned to 180 degrees
- moved R14 280.7 mm to (-120.2, 117.7), turned to -90 degrees
- moved R_CHG_MG2 280.5 mm to (-131.6, 43.1), turned to 180 degrees
- moved R_CHG_MG1 280.0 mm to (-131.6, 38.9)
- moved R_MID1 279.4 mm to (-109.6, 98.0), turned to 90 degrees
- moved C20 279.2 mm to (-118.6, 117.7), turned to 90 degrees
- moved R_PACK_FLT1 276.8 mm to (-106.4, 98.0), turned to 90 degrees
- moved D_CHG_VGS1 276.3 mm to (-127.4, 40.5), turned to 0 degrees
- moved R15 275.3 mm to (-115.0, 117.7), turned to -90 degrees
- moved U11 274.3 mm to (-110.9, 105.8), turned to 0 degrees
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Connections:
- C10 pad 2: +1V1 -> +3V3
- C11 pad 2: +3V3 -> +1V1
- C16 pad 1: GND -> +3V3
- C16 pad 2: +3V3 -> GND
- C21 pad 1: GND -> /main/BMS/NTC3
- C21 pad 2: /main/BMS/NTC3 -> GND
- C22 pad 1: GND -> /main/BMS/NTC2
- C22 pad 2: /main/BMS/NTC2 -> GND
- C23 pad 1: GND -> /main/BMS/NTC1
- C23 pad 2: /main/BMS/NTC1 -> GND
- C8 pad 1: /main/microcontroller/XR -> GND
- C8 pad 2: GND -> /main/microcontroller/XR
- C_PACK_FLT1 pad 1: GND -> Net-(U11-PACKP)
- C_PACK_FLT1 pad 2: Net-(U11-PACKP) -> GND
- C_SRN_GND1 pad 1: /main/BMS/SRN -> GND
- C_SRN_GND1 pad 2: GND -> /main/BMS/SRN
- C_SRP_GND1 pad 1: GND -> /main/BMS/SRP
- C_SRP_GND1 pad 2: /main/BMS/SRP -> GND
- J1 pad A6: /main/external_io/D+ -> /main/external_io/Dp
- J1 pad A7: /main/external_io/D- -> /main/external_io/Dn
- J1 pad B6: /main/external_io/D+ -> /main/external_io/Dp
- J1 pad B7: /main/external_io/D- -> /main/external_io/Dn
- J2 pad 1: GND -> /main/BMS/PACK+
- J2 pad 2: Net-(J2-Pin_2) -> /main/BMS/PACK-
- J4 pad 1: /main/BMS/PACK+ -> GND
- J4 pad 2: /main/BMS/PACK- -> Net-(J4-Pin_2)
- J5 pad 1: /main/external_io/RX -> /main/external_io/BOOT
- J5 pad 2: /main/external_io/TX -> GND
- J5 pad 3: /main/external_io/BOOT -> /main/external_io/RUN
- J6 pad 1: /main/external_io/SWDIO -> /main/external_io/RX
- J6 pad 2: GND -> /main/external_io/TX
- J6 pad 3: /main/external_io/SWCLK -> GND
- J7 pad 1: /main/BMS/C5 -> /main/external_io/SWCLK
- J7 pad 2: /main/BMS/NTC1 -> GND
- J7 pad 3: /main/BMS/C4 -> /main/external_io/SWDIO
- J8 pad 1: GND -> /main/BMS/C5
- J8 pad 2: /main/BMS/TOP -> /main/BMS/C5
- J9 pad 1: unconnected-(J9-Pin_1-Pad1) -> GND
- J9 pad 2: unconnected-(J9-Pin_2-Pad2) -> /main/BMS/TOP
- R10 pad 1: /main/microcontroller/D+ -> /main/microcontroller/QSPI_SS
- R10 pad 2: /main/external_io/D+ -> /main/external_io/BOOT
- R11 pad 1: /main/microcontroller/D- -> /main/microcontroller/D+
- R11 pad 2: /main/external_io/D- -> /main/external_io/D+
- R12 pad 1: +3V3 -> /main/external_io/D-
- R12 pad 2: Net-(U3-VREG_AVDD) -> /main/microcontroller/D-
- R13 pad 1: /main/BMS/NTC4 -> +3V3
- R13 pad 2: Net-(U11-NTCB) -> Net-(U3-VREG_AVDD)
- R14 pad 1: /main/BMS/NTC3 -> /main/BMS/NTC4
- R15 pad 1: /main/BMS/NTC2 -> /main/BMS/NTC3
- R16 pad 1: /main/BMS/NTC1 -> GND
- R16 pad 2: Net-(U11-NTCB) -> /main/BMS/NTC1
- R17 pad 1: /main/BMS/nSHDN -> GND
- R17 pad 2: +3V3 -> /main/BMS/NTC2
- R3 pad 1: /main/external_io/SWCLK -> GND
- R3 pad 2: /main/microcontroller/SWCLK_INT -> /main/BMS/nSHDN
- R4 pad 1: /main/microcontroller/SWDIO_INT -> GND
- R4 pad 2: /main/external_io/SWDIO -> /main/BMS/SDA
- R5 pad 1: GND -> /main/BMS/SCL
- R5 pad 2: /main/BMS/SDA -> GND
- R6 pad 1: /main/BMS/SCL -> /main/external_io/SWCLK
- R6 pad 2: GND -> /main/microcontroller/SWCLK_INT
- R7 pad 1: /main/external_io/RUN -> /main/microcontroller/SWDIO_INT
- R7 pad 2: Net-(U3-RUN) -> /main/external_io/SWDIO
- R8 pad 1: /main/microcontroller/XOUT -> /main/external_io/RUN
- R8 pad 2: /main/microcontroller/XR -> Net-(U3-RUN)
- R9 pad 1: /main/microcontroller/QSPI_SS -> /main/microcontroller/XOUT
- R9 pad 2: /main/external_io/BOOT -> /main/microcontroller/XR
- R_CELL_FLT1 pad 1: /main/BMS/TOP -> /main/BMS/CELL_6
- R_CELL_FLT1 pad 2: /main/BMS/CELL_6 -> /main/BMS/TOP
- R_CELL_FLT2 pad 1: /main/BMS/C5 -> /main/BMS/CELL_5
- R_CELL_FLT2 pad 2: /main/BMS/CELL_5 -> /main/BMS/C5
- R_CELL_FLT3 pad 1: /main/BMS/C4 -> /main/BMS/CELL_4
- R_CELL_FLT3 pad 2: /main/BMS/CELL_4 -> /main/BMS/C4
- R_CELL_FLT4 pad 1: /main/BMS/C3 -> /main/BMS/CELL_3
- R_CELL_FLT4 pad 2: /main/BMS/CELL_3 -> /main/BMS/C3
- R_CELL_FLT5 pad 1: /main/BMS/C2 -> /main/BMS/CELL_2
- R_CELL_FLT5 pad 2: /main/BMS/CELL_2 -> /main/BMS/C2
- R_CELL_FLT6 pad 1: /main/BMS/C1 -> /main/BMS/CELL_1
- R_CELL_FLT6 pad 2: /main/BMS/CELL_1 -> /main/BMS/C1
- R_CELL_FLT7 pad 1: GND -> /main/BMS/CELL_0
- R_CELL_FLT7 pad 2: /main/BMS/CELL_0 -> GND
- R_CHG_MG1 pad 1: Net-(D_CHG_VGS1-K) -> Net-(Q2-G)
- R_CHG_MG1 pad 2: Net-(Q2-G) -> Net-(D_CHG_VGS1-K)
- R_DSG_DRIVER1 pad 1: /main/BMS/DSG -> Net-(D_CHG_VGS2-K)
- R_DSG_DRIVER1 pad 2: Net-(D_CHG_VGS2-K) -> /main/BMS/DSG
- R_DSG_MG1 pad 1: Net-(D_CHG_VGS2-K) -> Net-(Q5-G)
- R_DSG_MG1 pad 2: Net-(Q5-G) -> Net-(D_CHG_VGS2-K)
- R_DSG_MG2 pad 1: Net-(Q4-G) -> Net-(D_CHG_VGS2-K)
- R_DSG_MG2 pad 2: Net-(D_CHG_VGS2-K) -> Net-(Q4-G)
- R_MID1 pad 1: /main/BMS/DRAIN -> Net-(U11-VMID)
- R_MID1 pad 2: Net-(U11-VMID) -> /main/BMS/DRAIN
- TP1 pad 1: /main/BMS/CELL_6 -> /main/BMS/XALERT
- TP2 pad 1: /main/BMS/CELL_5 -> /main/BMS/WDT
- TP3 pad 1: /main/BMS/CELL_4 -> /main/BMS/nSHDN
- TP4 pad 1: /main/BMS/CELL_3 -> /main/BMS/CELL_6
- TP5 pad 1: /main/BMS/CELL_2 -> /main/BMS/CELL_5
- TP6 pad 1: /main/BMS/CELL_1 -> /main/BMS/CELL_4
- TP7 pad 1: /main/BMS/CELL_0 -> /main/BMS/CELL_3
- U1 pad 1: Net-(J2-Pin_2) -> /main/external_io/Dp
- U1 pad 3: Net-(J2-Pin_3) -> /main/external_io/Dn
- U1 pad 4: /main/BMS/SCL -> /main/external_io/D-
- U1 pad 5: /main/EXT_5V -> /main/V_USB
- U1 pad 6: /main/BMS/SDA -> /main/external_io/D+
- U2 pad 1: /main/external_io/D+ -> Net-(J4-Pin_2)
- U2 pad 3: /main/external_io/D- -> Net-(J4-Pin_3)
- U2 pad 4: /main/external_io/D- -> /main/BMS/SCL
- U2 pad 5: unconnected-(U2-VBUS-Pad5) -> /main/EXT_5V
- U2 pad 6: /main/external_io/D+ -> /main/BMS/SDA
- U3 pad 12: GND -> unconnected-(U3-GPIO8-Pad12)
- U3 pad 13: GND -> unconnected-(U3-GPIO9-Pad13)
- U3 pad 15: /main/microcontroller/nSHDN -> /main/BMS/nSHDN
- U3 pad 17: GND -> unconnected-(U3-GPIO13-Pad17)
- U3 pad 18: GND -> unconnected-(U3-GPIO14-Pad18)
- U3 pad 19: GND -> unconnected-(U3-GPIO15-Pad19)
- U3 pad 7: GND -> unconnected-(U3-GPIO4-Pad7)
- U3 pad 8: GND -> unconnected-(U3-GPIO5-Pad8)
- U4 pad 3: GND -> unconnected-(U4-NC-Pad3)
- U4 pad 5: unconnected-(U4-DNC-Pad5) -> GND
- U4 pad 6: +3V3 -> GND
- U4 pad 7: GND -> unconnected-(U4-NC-Pad7)
- U4 pad 8: (no net) -> +3V3
Routing:
- net +3V3: track 81.9 -> 0.00 mm, vias 8 -> 0
- net /main/external_io/D-: track 62.6 -> 0.00 mm
- net Net-(D_CHG_VGS2-K): track 61.0 -> 0.00 mm, vias 2 -> 0
- net /main/external_io/D+: track 60.6 -> 0.00 mm
- net /main/BMS/NSHDN: track 53.9 -> 0.00 mm, vias 2 -> 0
- net Net-(D_CHG_VGS1-K): track 50.1 -> 0.00 mm, vias 2 -> 0
- net +1V1: track 49.3 -> 0.00 mm, vias 3 -> 0
- net /main/BMS/SCL: track 48.4 -> 0.00 mm, vias 4 -> 0
- net /main/INT_5V: track 45.3 -> 0.00 mm, vias 2 -> 0
- net /main/BMS/CELL_5: track 45.1 -> 0.00 mm, vias 2 -> 0
- net /main/BMS/SDA: track 44.4 -> 0.00 mm, vias 4 -> 0
- net /main/BMS/TOP: track 42.5 -> 0.00 mm, vias 3 -> 0
- net /main/external_io/SWCLK: track 40.2 -> 0.00 mm, vias 2 -> 0
- net /main/external_io/SWDIO: track 40.1 -> 0.00 mm, vias 2 -> 0
- net /main/EXT_5V: track 39.7 -> 0.00 mm, vias 3 -> 0
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- removed copper zone on B.Cu, net +1V1
- removed copper zone on B.Cu, net +3V3
- removed copper zone on B.Cu, net /main/BMS/C10
- removed copper zone on B.Cu, net /main/BMS/CELL_6
- removed copper zone on F.Cu, net /main/BMS/DRAIN
- removed copper zone on B.Cu, net /main/BMS/PACK+
- removed copper zone on F.Cu, net /main/BMS/PACK+
- removed copper zone on In1.Cu, net /main/BMS/PACK+
- removed copper zone on B.Cu, net /main/BMS/PACK-
- removed copper zone on F.Cu, net /main/BMS/PACK-
- removed copper zone on F.Cu, net /main/BMS/TOP
- removed copper zone on B.Cu, net /main/housekeeping/5V_IN
- removed copper zone on B.Cu, net GND
- removed copper zone on F.Cu, net GND
- removed copper zone on In1.Cu, net GND
- removed copper zone on In2.Cu, net GND
- removed copper zone on In3.Cu, net GND
- removed copper zone on In4.Cu, net GND
- removed copper zone on B.Cu, net Net-(D_CHG_VGS1-K)
- removed copper zone on F.Cu, net Net-(R_BAL_1-Pad1)
- removed copper zone on F.Cu, net Net-(R_BAL_2-Pad1)
- removed copper zone on F.Cu, net Net-(R_BAL_3-Pad1)
- removed copper zone on F.Cu, net Net-(R_BAL_4-Pad1)
- removed copper zone on F.Cu, net Net-(R_BAL_5-Pad1)
- removed copper zone on F.Cu, net Net-(R_BAL_6-Pad1)
- removed copper zone on B.Cu, net Net-(U3-VREG_LX)
Other:
- board outline removed
- board text removed: "Alejandro A."
- board text removed: "Ezzat S."

Commit message: Doing placement
Parts:
- removed J3: Conn_01x02_Socket, Connector_AMASS:AMASS_XT30PW-F_1x02_P2.50mm_Horizontal
- added D12: LED, LED_SMD:LED_0603_1608Metric, F.Cu at (240.1, 70.3)
- added D13: LED, LED_SMD:LED_0603_1608Metric, F.Cu at (234.1, 58.2)
- added D14: LED, LED_SMD:LED_0603_1608Metric, F.Cu at (234.1, 60.8)
- added D15: LED, LED_SMD:LED_0603_1608Metric, F.Cu at (244.1, 58.2)
- added D16: LED, LED_SMD:LED_0603_1608Metric, F.Cu at (244.1, 60.8)
- added D17: LED, LED_SMD:LED_0603_1608Metric, F.Cu at (244.1, 63.4)
- added R22: R, Resistor_SMD:R_0603_1608Metric, F.Cu at (244.1, 72.8)
- added R23: R, Resistor_SMD:R_0603_1608Metric, F.Cu at (234.0, 63.4)
- added R24: R, Resistor_SMD:R_0603_1608Metric, F.Cu at (234.0, 65.9)
- added R25: R, Resistor_SMD:R_0603_1608Metric, F.Cu at (240.1, 60.7)
- added R26: R, Resistor_SMD:R_0603_1608Metric, F.Cu at (240.1, 63.2)
- added R27: R, Resistor_SMD:R_0603_1608Metric, F.Cu at (240.1, 65.7)
- added TP11: TestPoint, TestPoint:TestPoint_Pad_D2.0mm, F.Cu at (240.1, 73.6)
- added TP12: TestPoint, TestPoint:TestPoint_Pad_D2.0mm, F.Cu at (230.0, 59.0)
- added TP13: TestPoint, TestPoint:TestPoint_Pad_D2.0mm, F.Cu at (230.0, 63.0)
- C1, C10, C11, C12, C13, C14, C15, C16, C17, C18, C2, C20, C21, C22, C23, C3, C4, C5, C6, C7, C8, C9, C_3V3_1, C_CELL_FLT1, C_CELL_FLT2, C_CELL_FLT3, C_CELL_FLT4, C_CELL_FLT5, C_CELL_FLT6, C_CP1, C_MID1, C_PACK_FLT1, C_REG1, C_REGIN1, C_SRN_GND1, C_SRP_GND1, C_SRP_SRN1, C_TOP_FLT1, C_VDD1, C_VREF1, D1, D2, D3, J4, L1, Q1, R11, R12, R13, R14, R15, R16, R17, R18, R19, R20, R21, R3, R4, R5, R6, R7, R9, R_MID1, R_PACK_FLT1, R_REG1, R_SRN_FLT1, R_SRP_FLT1, R_TOP_FLT1, U11, U3, U4, X1: moved to B.Cu
- J10, J11, J12, J13: footprint Connector_JST:JST_PH_S2B-PH-SM4-TB_1x02-1MP_P2.00mm_Horizontal -> Connector_JST:JST_GH_SM02B-GHS-TB_1x02-1MP_P1.25mm_Horizontal; moved to B.Cu
- R10: value 1k -> 10k; moved to B.Cu
- R8: value 1k -> 10k
- moved R14 285.3 mm to (160.0, 63.7), turned to 0 degrees
- moved C20 283.5 mm to (160.0, 65.3), turned to 180 degrees
- moved R19 281.6 mm to (160.0, 66.9), turned to 180 degrees
- moved R15 279.3 mm to (160.0, 68.9), turned to 0 degrees
- moved C21 277.4 mm to (160.0, 70.5), turned to 0 degrees
- moved R_SRP_FLT1 275.8 mm to (156.0, 67.9), turned to 180 degrees
- moved R18 275.6 mm to (160.0, 72.1), turned to 180 degrees
- moved C_CELL_FLT6 274.3 mm to (152.1, 65.3), turned to -90 degrees
- moved C_SRP_GND1 274.0 mm to (156.0, 69.5), turned to 0 degrees
- moved R20 273.3 mm to (160.0, 74.1), turned to 0 degrees
- moved C_CELL_FLT5 272.5 mm to (150.5, 65.3), turned to -90 degrees
- moved R_CHG_PUP1 272.2 mm to (140.3, 54.5), turned to -90 degrees
- moved C22 271.4 mm to (160.0, 75.7), turned to 0 degrees
- moved C_SRP_SRN1 271.4 mm to (156.0, 71.8), turned to 90 degrees
- moved C_CELL_FLT4 270.6 mm to (148.9, 65.3), turned to 90 degrees
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Connections:
- R10 pad 1: /main/microcontroller/QSPI_SS -> +3V3
- R3 pad 1: GND -> +3V3
- R4 pad 1: GND -> +3V3
- R5 pad 2: GND -> +3V3
- R8 pad 2: Net-(U3-RUN) -> +3V3
- U3 pad 26: Net-(U3-RUN) -> +3V3
- U3 pad 31: unconnected-(U3-GPIO19-Pad31) -> +3V3
- U3 pad 32: unconnected-(U3-GPIO20-Pad32) -> +3V3
- U3 pad 33: unconnected-(U3-GPIO21-Pad33) -> +3V3
- U3 pad 60: /main/microcontroller/QSPI_SS -> +3V3
Routing:
- net /main/microcontroller/XIN: track 0.00 -> 5.67 mm
Other:
- board outline added: 67 x 60 mm

Commit message: Prelim placement done
Parts:
- removed D12: LED, LED_SMD:LED_0603_1608Metric
- removed J2: Conn_01x02_Socket, Connector_AMASS:AMASS_XT30PW-F_1x02_P2.50mm_Horizontal
- removed R22: R, Resistor_SMD:R_0603_1608Metric
- removed TP11, TP12, TP13: TestPoint, TestPoint:TestPoint_Pad_D2.0mm
- added H3: MountingHole, MountingHole:MountingHole_2.2mm_M2_Pad_TopBottom, F.Cu at (169.0, 59.0)
- added H4: MountingHole, MountingHole:MountingHole_2.2mm_M2_Pad_TopBottom, F.Cu at (169.0, 121.0)
- added J3: Conn_01x02_Socket, Connector_AMASS:AMASS_XT30PW-F_1x02_P2.50mm_Horizontal, F.Cu at (118.8, 92.5)
- C19, C_PACK_E1, C_PACK_E2, C_PACK_E3, D11, R8, U2: moved to B.Cu
- R_CHG_PUP1, R_DSG_PUP1: footprint Resistor_SMD:R_0402_1005Metric -> Resistor_SMD:R_0603_1608Metric; moved to B.Cu
- U10, U5, U6, U7, U8, U9: footprint _BMS:SC70-6 -> _BMS:SC_4EEH-T1_GE3_VIS
- moved C19 198.6 mm to (167.3, 75.3)
- moved L1 149.3 mm to (119.1, 70.9), turned to 90 degrees
- moved R12 148.9 mm to (120.7, 66.7)
- moved R11 148.1 mm to (120.7, 68.3), turned to 180 degrees
- moved C15 146.8 mm to (120.8, 70.9), turned to 90 degrees
- moved C16 144.3 mm to (122.4, 70.9), turned to -90 degrees
- moved C_PACK_E1 141.1 mm to (113.8, 92.9)
- moved C_PACK_E2 138.9 mm to (113.8, 90.3)
- moved C14 138.4 mm to (121.6, 74.3), turned to 180 degrees
- moved C13 138.3 mm to (124.6, 75.4), turned to 90 degrees
- moved R13 137.1 mm to (121.6, 75.9), turned to 0 degrees
- moved C_PACK_E3 136.9 mm to (113.8, 87.8)
- moved U3 135.9 mm to (127.4, 69.1), turned to -90 degrees
- moved C12 135.4 mm to (126.2, 75.4), turned to -90 degrees
- moved C11 132.0 mm to (129.4, 75.4), turned to 90 degrees
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Routing:
- net /main/microcontroller/XOUT: track 0.00 -> 5.98 mm
- net /main/microcontroller/XIN: track 5.67 -> 10.7 mm
- net /main/microcontroller/XR: track 0.00 -> 3.59 mm
- net +1V1: track 0.00 -> 2.71 mm
- net +3V3: track 0.00 -> 2.68 mm
Other:
- board size 67 x 60 mm -> 64 x 70 mm

Commit message: Did a lot of routing
Parts:
- D_CHG_VGS1, D_CHG_VGS2, R_CHG_DRIVER1, R_CHG_MG1, R_CHG_MG2, R_CHG_PUP1, R_DSG_DRIVER1, R_DSG_MG1, R_DSG_MG2, R_DSG_PUP1: moved to F.Cu
- J1, R1, R2, U1: moved to B.Cu
- L1: footprint Inductor_SMD:L_0805_2012Metric -> _BMS:rp_inductor
- TP1, TP2, TP3: footprint TestPoint:TestPoint_Keystone_5015_Micro_Mini -> _BMS:Harwin TP
- moved J4 74.8 mm to (114.1, 113.0), turned to 90 degrees
- moved U2 66.3 mm to (120.0, 113.0), turned to 0 degrees
- moved J6 54.5 mm to (149.5, 62.6)
- moved J7 54.5 mm to (159.0, 62.6)
- moved J5 53.9 mm to (125.4, 62.2), turned to -90 degrees
- moved R14 46.4 mm to (164.1, 111.0), turned to 180 degrees
- moved R4 45.3 mm to (122.9, 114.8), turned to 90 degrees
- moved U1 43.3 mm to (121.3, 70.4), turned to 0 degrees
- moved C20 43.2 mm to (164.1, 109.4)
- moved R1 41.9 mm to (120.8, 66.3)
- moved R_SRP_FLT1 40.9 mm to (129.2, 95.4), turned to 0 degrees
- moved C17 40.5 mm to (123.5, 76.0)
- moved R5 40.4 mm to (122.9, 111.2), turned to 90 degrees
- moved R19 40.0 mm to (164.1, 107.8), turned to 0 degrees
- moved C19 39.6 mm to (129.2, 86.0)
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Routing:
- net +3V3: track 2.68 -> 111.2 mm, vias 0 -> 10
- net Net-(U11-NTCB): track 0.00 -> 91.2 mm, vias 0 -> 6
- net /main/BMS/SDA: track 0.00 -> 79.5 mm, vias 0 -> 4
- net /main/BMS/SCL: track 0.00 -> 74.8 mm, vias 0 -> 4
- net /main/BMS/C5: track 0.00 -> 67.5 mm, vias 0 -> 5
- net /main/BMS/NTC3: track 0.00 -> 60.7 mm, vias 0 -> 2
- net /main/BMS/C4: track 0.00 -> 58.6 mm, vias 0 -> 5
- net /main/BMS/CELL_5: track 0.00 -> 58.3 mm, vias 0 -> 1
- net /main/BMS/NTC4: track 0.00 -> 56.1 mm, vias 0 -> 2
- net /main/BMS/CELL_0: track 0.00 -> 54.0 mm, vias 0 -> 1
- net /main/BMS/CELL_4: track 0.00 -> 52.5 mm, vias 0 -> 1
- net /main/BMS/TOP: track 0.00 -> 52.0 mm, vias 0 -> 33
- net /main/BMS/C3: track 0.00 -> 51.2 mm, vias 0 -> 5
- net /main/BMS/NTC1: track 0.00 -> 50.3 mm, vias 0 -> 2
- net /main/BMS/NTC2: track 0.00 -> 50.1 mm, vias 0 -> 2
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- added copper zone on B.Cu, net +1V1
- added copper zone on B.Cu, net +3V3
- added copper zone on In3.Cu, net +3V3
- added copper zone on F.Cu, net /main/BMS/DRAIN
- added copper zone on F.Cu, net /main/BMS/PACK+
- added copper zone on In2.Cu, net /main/BMS/PACK+
- added copper zone on F.Cu, net /main/BMS/PACK-
- added copper zone on F.Cu, net /main/BMS/TOP
- added copper zone on In2.Cu, net /main/BMS/TOP
- added copper zone on B.Cu, net GND
- added copper zone on F.Cu, net GND
- added copper zone on In1.Cu, net GND
- added copper zone on In2.Cu, net GND
- added copper zone on In3.Cu, net GND
- added copper zone on In4.Cu, net GND
- added copper zone on F.Cu, net Net-(R_BAL_1-Pad1)
- added copper zone on F.Cu, net Net-(R_BAL_2-Pad1)
- added copper zone on F.Cu, net Net-(R_BAL_3-Pad1)
- added copper zone on F.Cu, net Net-(R_BAL_4-Pad1)
- added copper zone on F.Cu, net Net-(R_BAL_5-Pad1)
- added copper zone on F.Cu, net Net-(R_BAL_6-Pad1)
- added copper zone on B.Cu, net Net-(U3-VREG_LX)
Other:
- board size 64 x 70 mm -> 64.6 x 70 mm

Commit message: Working on routing
Parts:
- moved R8 41.7 mm to (157.6, 65.3), turned to -90 degrees
- moved J5 37.3 mm to (162.7, 62.3)
- moved J6 26.4 mm to (123.0, 61.9)
- moved R3 22.8 mm to (138.6, 61.9), turned to -90 degrees
- moved J7 10.2 mm to (148.8, 62.3)
- moved R6 1.60 mm to (145.4, 61.5)
- moved R7 1.60 mm to (145.4, 63.1)
- turned D15 to -90 degrees
- turned D16 to -90 degrees
- turned D17 to -90 degrees
- turned R25 to 90 degrees
- turned R26 to 90 degrees
- turned R27 to 90 degrees
- turned R_CHG_PUP1 to -90 degrees
Connections:
- D15 pad 1: Net-(D15-K) -> GND
- D15 pad 2: +3V3 -> /main/microcontroller/LED1
- D16 pad 1: Net-(D16-K) -> GND
- D16 pad 2: +3V3 -> /main/microcontroller/LED2
- D17 pad 1: Net-(D17-K) -> GND
- D17 pad 2: +3V3 -> /main/microcontroller/LED3
- R25 pad 1: Net-(D15-K) -> +3V3
- R25 pad 2: GND -> /main/microcontroller/LED1
- R26 pad 1: Net-(D16-K) -> +3V3
- R26 pad 2: GND -> /main/microcontroller/LED2
- R27 pad 1: Net-(D17-K) -> +3V3
- R27 pad 2: GND -> /main/microcontroller/LED3
- R_CHG_PUP1 pad 1: Net-(D_CHG_VGS1-K) -> /main/BMS/TOP
- R_CHG_PUP1 pad 2: /main/BMS/TOP -> Net-(D_CHG_VGS1-K)
- U3 pad 31: +3V3 -> /main/microcontroller/LED3
- U3 pad 32: +3V3 -> /main/microcontroller/LED2
- U3 pad 33: +3V3 -> /main/microcontroller/LED1
Routing:
- net /main/BMS/TOP: track 52.0 -> 18.4 mm, vias 33 -> 34
- net /main/external_io/BOOT: track 0.00 -> 32.7 mm, vias 0 -> 1
- net +3V3: track 111.2 -> 86.1 mm, vias 10 -> 9
- net +1V1: track 31.8 -> 7.93 mm, vias 5 -> 0
- net /main/external_io/RX: track 0.00 -> 14.1 mm, vias 0 -> 1
- net /main/microcontroller/SWCLK_INT: track 0.00 -> 11.6 mm, vias 0 -> 2
- net /main/external_io/TX: track 0.00 -> 11.0 mm, vias 0 -> 1
- net /main/microcontroller/SWDIO_INT: track 0.00 -> 10.7 mm, vias 0 -> 2
- net /main/external_io/SWDIO: track 0.00 -> 8.35 mm
- net GND: track 2.36 -> 5.56 mm, vias 1 -> 0
- net /main/external_io/SWCLK: track 0.00 -> 2.88 mm
- net /main/BMS/PACK+: track 37.4 -> 39.8 mm
- net /main/external_io/RUN: track 0.00 -> 2.18 mm
- net Net-(D14-A): track 0.00 -> 1.62 mm
- net Net-(D16-K): track 1.49 -> 0.00 mm
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