File: BMS.kicad_pcb (KiCad board)
At the start: 6 copper layers, 65 x 70 mm, 190 parts, among them J1 UJ20-C-H-G-SMT-1-P16-TR, J10 Conn_01x02_Pin, J11 Conn_01x02_Pin, J12 Conn_01x03_Socket, J2 Conn_01x02_Socket, J3 Conn_01x03_Socket, J4 Conn_01x04_Socket, J5 Conn_01x03_Socket, J6 Conn_01x03_Socket, J7 Conn_01x10_Pin, J8 Conn_01x02_Pin, J9 Conn_01x02_Pin, Q1 FZT853TA, Q2 PSMN3R7-100BSE, Q3 PSMN3R7-100BSE, Q4 PSMN3R7-100BSE, Q5 PSMN3R7-100BSE, Q6 Q_PMOS_GDS, U1 USBLC6-2SC6, U10 SQ1464EEH-T1_GE3, U11 MP2790DFP-0000-T, U2 W25Q64JVSSIQ, U3 RP2350A, U4 TPS7B8133QDGNRQ1, U5 SQ1464EEH-T1_GE3, U6 SQ1464EEH-T1_GE3, U7 SQ1464EEH-T1_GE3, U8 SQ1464EEH-T1_GE3, U9 SQ1464EEH-T1_GE3, X1 ABM8-272-T3

Commit message: Pushing
Parts:
- R31: value R -> 1k
