File: BMS.kicad_pcb (KiCad board)
At the start: 6 copper layers, 65 x 70 mm, 190 parts, among them J1 UJ20-C-H-G-SMT-1-P16-TR, J10 Conn_01x02_Pin, J11 Conn_01x02_Pin, J12 Conn_01x03_Socket, J2 Conn_01x02_Socket, J3 Conn_01x03_Socket, J4 Conn_01x04_Socket, J5 Conn_01x03_Socket, J6 Conn_01x03_Socket, J7 Conn_01x10_Pin, J8 Conn_01x02_Pin, J9 Conn_01x02_Pin, Q1 FZT853TA, Q2 PSMN3R7-100BSE, Q3 PSMN3R7-100BSE, Q4 PSMN3R7-100BSE, Q5 PSMN3R7-100BSE, Q6 Q_PMOS_GDS, U1 USBLC6-2SC6, U10 SQ1464EEH-T1_GE3, U11 MP2790DFP-0000-T, U2 W25Q64JVSSIQ, U3 RP2350A, U4 TPS7B8133QDGNRQ1, U5 SQ1464EEH-T1_GE3, U6 SQ1464EEH-T1_GE3, U7 SQ1464EEH-T1_GE3, U8 SQ1464EEH-T1_GE3, U9 SQ1464EEH-T1_GE3, X1 ABM8-272-T3

Commit message: Adding in JST XH
Parts:
- removed J7: Conn_01x10_Pin, _BMS:TB4-Hirose
- removed R10, R11: 33k, Resistor_SMD:R_0603_1608Metric
- removed U1: USBLC6-2SC6, Package_TO_SOT_SMD:SOT-23-6
- added C104: 18pF, Capacitor_SMD:C_0603_1608Metric, B.Cu at (131.1, 98.3)
- added C105: 18pF, Capacitor_SMD:C_0603_1608Metric, B.Cu at (131.1, 93.3)
- added C106: 47pF, Capacitor_SMD:C_0603_1608Metric, B.Cu at (117.7, 93.7)
- added C107: 47pF, Capacitor_SMD:C_0603_1608Metric, B.Cu at (117.7, 98.6)
- added D27: AQ24C-01FTG, Diode_SMD:D_0805_2012Metric, B.Cu at (117.9, 92.0)
- added D28: AQ24C-01FTG, Diode_SMD:D_0805_2012Metric, B.Cu at (117.9, 96.9)
- added J13: Conn_01x07_Pin, Connector_JST:JST_XH_S7B-XH-A-1_1x07_P2.50mm_Horizontal, F.Cu at (167.3, 111.1)
- added JP1: SolderJumper_2_Open, Jumper:SolderJumper-2_P1.3mm_Open_RoundedPad1.0x1.5mm, F.Cu at (111.3, 98.0)
- added R94: 10K, Resistor_SMD:R_0603_1608Metric, B.Cu at (121.2, 97.7)
- added R95: 10K, Resistor_SMD:R_0603_1608Metric, B.Cu at (120.0, 94.5)
- added R97: 120, Resistor_SMD:R_0603_1608Metric, B.Cu at (117.7, 95.2)
- added U19: MCP25625-E/ML, _BMS:QFN-28L, B.Cu at (125.2, 94.5)
- added Y1: 16MHz 12pF, Crystal:Crystal_SMD_2520-4Pin_2.5x2.0mm, B.Cu at (131.1, 95.8)
- moved FB2 17.2 mm to (135.0, 97.2), turned to 0 degrees
- moved C11 1.36 mm to (116.9, 100.2), turned to 0 degrees
- moved J11 0.70 mm to (171.2, 97.0)
- moved J9 0.70 mm to (171.2, 112.0)
- moved J10 0.65 mm to (171.2, 104.5)
- moved C22 0.20 mm to (164.7, 97.0)
- moved C23 0.20 mm to (164.7, 104.5)
- moved R25 0.20 mm to (164.7, 98.6)
- moved R27 0.20 mm to (164.7, 102.9)
- moved R28 0.20 mm to (164.7, 95.4)
- moved R30 0.20 mm to (164.7, 106.1)
- moved C24 0.15 mm to (164.7, 112.0)
- moved R26 0.15 mm to (164.7, 110.4)
- moved R32 0.15 mm to (164.7, 113.6)
- moved C20 0.10 mm to (161.7, 101.3)
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Connections:
- net Net-(D6-K) renamed +5V
- FB2 pad 2: Net-(J4-Pin_4) -> Net-(J4-Pin_1)
- J4 pad 1: GND -> Net-(J4-Pin_1)
- J4 pad 2: Net-(J4-Pin_2) -> /main/CAN/CANH
- J4 pad 3: Net-(J4-Pin_3) -> /main/CAN/CANL
- J4 pad 4: Net-(J4-Pin_4) -> GND
- R4 pad 1: Net-(J4-Pin_4) -> Net-(J4-Pin_1)
- U3 pad 12: unconnected-(U3-GPIO8-Pad12) -> /main/CAN/CS
- U3 pad 13: unconnected-(U3-GPIO9-Pad13) -> /main/CAN/CAN_RESET
- U3 pad 34: /main/external_io/SDA -> unconnected-(U3-GPIO22-Pad34)
- U3 pad 35: /main/external_io/SCL -> unconnected-(U3-GPIO23-Pad35)
- U3 pad 4: unconnected-(U3-GPIO2-Pad4) -> /main/CAN/SCK
- U3 pad 5: unconnected-(U3-GPIO3-Pad5) -> /main/CAN/MOSI
- U3 pad 7: unconnected-(U3-GPIO4-Pad7) -> /main/CAN/MISO
- U3 pad 8: unconnected-(U3-GPIO5-Pad8) -> /main/CAN/CAN_INT
Routing:
- net Net-(J4-Pin_1): track 0.00 -> 39.2 mm, vias 0 -> 2
- net /main/external_io/SCL: track 35.4 -> 0.00 mm, vias 2 -> 0
- net /main/external_io/SDA: track 34.0 -> 0.00 mm, vias 2 -> 0
- net /main/CAN/CANH: track 0.00 -> 32.2 mm, vias 0 -> 1
- net /main/BMS/TOP: track 143.2 -> 166.0 mm, vias 56 -> 55
- net /main/CAN/CAN_RESET: track 0.00 -> 20.4 mm, vias 0 -> 2
- net +3V3: track 62.7 -> 82.3 mm, vias 11 -> 14
- net /main/EXT_5V: track 20.6 -> 1.41 mm
- net /main/CAN/SCK: track 0.00 -> 19.1 mm, vias 0 -> 2
- net GND: track 24.0 -> 41.6 mm, vias 34 -> 39
- net /main/CAN/CANL: track 0.00 -> 16.6 mm
- net Net-(U19-TXCAN): track 0.00 -> 15.2 mm, vias 0 -> 2
- net /main/CAN/CS: track 0.00 -> 14.4 mm, vias 0 -> 2
- net /main/CAN/MISO: track 0.00 -> 13.6 mm, vias 0 -> 2
- net /main/CAN/CAN_INT: track 0.00 -> 13.3 mm
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- removed copper zone on F.Cu, net /main/BMS/C1
- removed copper zone on F.Cu, net /main/BMS/C2
- removed copper zone on F.Cu, net /main/BMS/C3
- removed copper zone on F.Cu, net /main/BMS/C4
- removed copper zone on F.Cu, net /main/BMS/C5
Other:
- board size 65 x 70 mm -> 65.5 x 70 mm
- board text added: "*"
- board text added: "CAN"
- board text removed: "I2C"
