File: bossmodeshi.kicad_sch (KiCad schematic)
At the start: 92 parts, among them Q1 FZT853TA, Q2 PSMN020-100YS, Q3 PSMN020-100YS, Q4 PSMN3R7-100BSE, Q5 PSMN3R7-100BSE, U10 SQ1464EEH-T1_GE3, U11 MP2790DFP-0000-T, U5 SQ1464EEH-T1_GE3, U6 SQ1464EEH-T1_GE3, U7 SQ1464EEH-T1_GE3, U8 SQ1464EEH-T1_GE3, U9 SQ1464EEH-T1_GE3

Commit message: Tweaks and production files
Parts:
- renumbered TP4 to TP1, TP5 to TP2, TP6 to TP3, TP7 to TP4, TP8 to TP5, TP9 to TP6, TP10 to TP7
Changed lines of the file:
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@@
 		(dnp no)
 		(fields_autoplaced yes)
-		(property "Reference" "#PWR061"
+		(property "Reference" "#PWR060"
 			(at 218.44 160.02 0)
 			(effects
@@
 			(project "BMS"
 				(path "/124184ba-5d68-4d9f-8da6-acc6720ab30b/93f9b420-7cce-46a9-9201-666f07a18f85/d98fdb38-dbd9-4613-8402-dc473e6cf2ba"
-					(reference "#PWR061")
+					(reference "#PWR060")
 					(unit 1)
 				)
@@
 		(dnp no)
 		(fields_autoplaced yes)
-		(property "Reference" "#PWR056"
+		(property "Reference" "#PWR054"
 			(at 156.21 119.38 0)
 			(effects
@@
 			(project "BMS"
 				(path "/124184ba-5d68-4d9f-8da6-acc6720ab30b/93f9b420-7cce-46a9-9201-666f07a18f85/d98fdb38-dbd9-4613-8402-dc473e6cf2ba"
-					(reference "#PWR056")
+					(reference "#PWR054")
 					(unit 1)
 				)
@@
 		(dnp no)
 		(fields_autoplaced yes)
-		(property "Reference" "#PWR054"
+		(property "Reference" "#PWR052"
 			(at 120.65 157.48 0)
 			(effects
@@
 			(project "BMS"
 				(path "/124184ba-5d68-4d9f-8da6-acc6720ab30b/93f9b420-7cce-46a9-9201-666f07a18f85/d98fdb38-dbd9-4613-8402-dc473e6cf2ba"
-					(reference "#PWR054")
+					(reference "#PWR052")
 					(unit 1)
 				)
@@
 		(dnp no)
 		(fields_autoplaced yes)
-		(property "Reference" "#PWR057"
+		(property "Reference" "#PWR055"
 			(at 156.21 196.85 0)
 			(effects
@@
 			(project "BMS"
 				(path "/124184ba-5d68-4d9f-8da6-acc6720ab30b/93f9b420-7cce-46a9-9201-666f07a18f85/d98fdb38-dbd9-4613-8402-dc473e6cf2ba"
-					(reference "#PWR057")
+					(reference "#PWR055")
 					(unit 1)
 				)
@@
 		(dnp no)
 		(fields_autoplaced yes)
-		(property "Reference" "TP7"
+		(property "Reference" "TP4"
 			(at 95.25 132.5879 0)
 			(effects
@@
 			(project "BMS"
 				(path "/124184ba-5d68-4d9f-8da6-acc6720ab30b/93f9b420-7cce-46a9-9201-666f07a18f85/d98fdb38-dbd9-4613-8402-dc473e6cf2ba"
-					(reference "TP7")
+					(reference "TP4")
 					(unit 1)
 				)
@@
 		(on_board yes)
 		(dnp no)
-		(property "Reference" "#PWR064"
+		(property "Reference" "#PWR062"
 			(at 313.69 130.81 0)
 			(effects
@@
 			(project "BMS"
 				(path "/124184ba-5d68-4d9f-8da6-acc6720ab30b/93f9b420-7cce-46a9-9201-666f07a18f85/d98fdb38-dbd9-4613-8402-dc473e6cf2ba"
-					(reference "#PWR064")
+					(reference "#PWR062")
 					(unit 1)
 				)
@@
 		(dnp no)
 		(fields_autoplaced yes)
-		(property "Reference" "TP5"
+		(property "Reference" "TP2"
 			(at 95.25 64.0079 0)
 			(effects
@@
 			(project "BMS"
 				(path "/124184ba-5d68-4d9f-8da6-acc6720ab30b/93f9b420-7cce-46a9-9201-666f07a18f85/d98fdb38-dbd9-4613-8402-dc473e6cf2ba"
-					(reference "TP5")
+					(reference "TP2")
 					(unit 1)
 				)
@@
 		(dnp no)
 		(fields_autoplaced yes)
-		(property "Reference" "TP9"
+		(property "Reference" "TP6"
 			(at 95.25 201.1679 0)
 			(effects
@@
 			(project "BMS"
 				(path "/124184ba-5d68-4d9f-8da6-acc6720ab30b/93f9b420-7cce-46a9-9201-666f07a18f85/d98fdb38-dbd9-4613-8402-dc473e6cf2ba"
-					(reference "TP9")
+					(reference "TP6")
 					(unit 1)
 				)
@@
 		(dnp no)
 		(fields_autoplaced yes)
-		(property "Reference" "TP8"
+		(property "Reference" "TP5"
 			(at 95.25 166.8779 0)
 			(effects
@@
 			(project "BMS"
 				(path "/124184ba-5d68-4d9f-8da6-acc6720ab30b/93f9b420-7cce-46a9-9201-666f07a18f85/d98fdb38-dbd9-4613-8402-dc473e6cf2ba"
-					(reference "TP8")
+					(reference "TP5")
 					(unit 1)
 				)
@@
 		(dnp no)
 		(fields_autoplaced yes)
-		(property "Reference" "#PWR067"
+		(property "Reference" "#PWR065"
 			(at 378.46 128.27 0)
 			(effects
@@
 			(project "BMS"
 				(path "/124184ba-5d68-4d9f-8da6-acc6720ab30b/93f9b420-7cce-46a9-9201-666f07a18f85/d98fdb38-dbd9-4613-8402-dc473e6cf2ba"
-					(reference "#PWR067")
+					(reference "#PWR065")
 					(unit 1)
 				)
@@
 		(dnp no)
 		(fields_autoplaced yes)
-		(property "Reference" "#PWR055"
+		(property "Reference" "#PWR053"
 			(at 138.43 149.86 0)
 			(effects
@@
 			(project ""
 				(path "/124184ba-5d68-4d9f-8da6-acc6720ab30b/93f9b420-7cce-46a9-9201-666f07a18f85/d98fdb38-dbd9-4613-8402-dc473e6cf2ba"
-					(reference "#PWR055")
+					(reference "#PWR053")
 					(unit 1)
 				)
@@
 		(dnp no)
 		(fields_autoplaced yes)
-		(property "Reference" "TP4"
+		(property "Reference" "TP1"
 			(at 95.25 29.7179 0)
 			(effects
@@
 			(project "BMS"
 				(path "/124184ba-5d68-4d9f-8da6-acc6720ab30b/93f9b420-7cce-46a9-9201-666f07a18f85/d98fdb38-dbd9-4613-8402-dc473e6cf2ba"
-					(reference "TP4")
+					(reference "TP1")
 					(unit 1)
 				)
@@
 		(dnp no)
 		(fields_autoplaced yes)
-		(property "Reference" "#PWR066"
+		(property "Reference" "#PWR064"
 			(at 356.87 144.78 0)
 			(effects
@@
 			(project "BMS"
 				(path "/124184ba-5d68-4d9f-8da6-acc6720ab30b/93f9b420-7cce-46a9-9201-666f07a18f85/d98fdb38-dbd9-4613-8402-dc473e6cf2ba"
-					(reference "#PWR066")
+					(reference "#PWR064")
 					(unit 1)
 				)
@@
 		(dnp no)
 		(fields_autoplaced yes)
-		(property "Reference" "#PWR062"
+		(property "Reference" "#PWR059"
 			(at 217.17 234.95 0)
 			(effects
@@
 			(project "BMS"
 				(path "/124184ba-5d68-4d9f-8da6-acc6720ab30b/93f9b420-7cce-46a9-9201-666f07a18f85/d98fdb38-dbd9-4613-8402-dc473e6cf2ba"
-					(reference "#PWR062")
+					(reference "#PWR059")
 					(unit 1)
 				)
@@
 		(dnp no)
 		(fields_autoplaced yes)
-		(property "Reference" "#PWR060"
+		(property "Reference" "#PWR057"
 			(at 176.53 256.54 0)
 			(effects
@@
 			(project "BMS"
 				(path "/124184ba-5d68-4d9f-8da6-acc6720ab30b/93f9b420-7cce-46a9-9201-666f07a18f85/d98fdb38-dbd9-4613-8402-dc473e6cf2ba"
-					(reference "#PWR060")
+					(reference "#PWR057")
 					(unit 1)
 				)
@@
 		(dnp no)
 		(fields_autoplaced yes)
-		(property "Reference" "#PWR065"
+		(property "Reference" "#PWR063"
 			(at 358.14 158.75 0)
 			(effects
@@
 			(project "BMS"
 				(path "/124184ba-5d68-4d9f-8da6-acc6720ab30b/93f9b420-7cce-46a9-9201-666f07a18f85/d98fdb38-dbd9-4613-8402-dc473e6cf2ba"
-					(reference "#PWR065")
+					(reference "#PWR063")
 					(unit 1)
 				)
@@
 		(dnp no)
 		(fields_autoplaced yes)
-		(property "Reference" "#PWR063"
+		(property "Reference" "#PWR061"
 			(at 246.38 234.95 0)
 			(effects
@@
 			(project "BMS"
 				(path "/124184ba-5d68-4d9f-8da6-acc6720ab30b/93f9b420-7cce-46a9-9201-666f07a18f85/d98fdb38-dbd9-4613-8402-dc473e6cf2ba"
-					(reference "#PWR063")
+					(reference "#PWR061")
 					(unit 1)
 				)
@@
 		(on_board yes)
 		(dnp no)
-		(property "Reference" "#PWR059"
+		(property "Reference" "#PWR056"
 			(at 176.53 45.72 0)
 			(effects
@@
 			(project "BMS"
 				(path "/124184ba-5d68-4d9f-8da6-acc6720ab30b/93f9b420-7cce-46a9-9201-666f07a18f85/d98fdb38-dbd9-4613-8402-dc473e6cf2ba"
-					(reference "#PWR059")
+					(reference "#PWR056")
 					(unit 1)
 				)
@@
 		(dnp no)
 		(fields_autoplaced yes)
-		(property "Reference" "TP10"
+		(property "Reference" "TP7"
 			(at 95.25 235.4579 0)
 			(effects
@@
 			(project "BMS"
 				(path "/124184ba-5d68-4d9f-8da6-acc6720ab30b/93f9b420-7cce-46a9-9201-666f07a18f85/d98fdb38-dbd9-4613-8402-dc473e6cf2ba"
-					(reference "TP10")
+					(reference "TP7")
 					(unit 1)
 				)
@@
 		(dnp no)
 		(fields_autoplaced yes)
-		(property "Reference" "TP6"
+		(property "Reference" "TP3"
 			(at 95.25 98.2979 0)
 			(effects
@@
 			(project "BMS"
 				(path "/124184ba-5d68-4d9f-8da6-acc6720ab30b/93f9b420-7cce-46a9-9201-666f07a18f85/d98fdb38-dbd9-4613-8402-dc473e6cf2ba"
-					(reference "TP6")
+					(reference "TP3")
 					(unit 1)
 				)

Commit message: Updating BOM
Parts:
- removed C_MID1: 100 nF, Capacitor_SMD:C_0402_1005Metric, symbol Device:C
- added C24: 100 nF, Capacitor_SMD:C_0402_1005Metric, symbol Device:C
- C_PACK_FLT1: Mfr KEMET -> YAGEO; Mfr P/N C0402C103J5RACAUTO -> AC0402JRX7R9BB103; Supplier_1 P/N 399-19365-2-ND -> 13-AC0402JRX7R9BB103TR-ND; Supplier_1 Unit Price 0.43000 -> 0.10000
- D11: Mfr Nexperia USA Inc. -> Vishay General Semiconductor - Diodes Division; Mfr P/N BAT46GWJ -> BAT46W-E3-18; Supplier_1 P/N 1727-7326-2-ND -> BAT46W-E3-18GITR-ND; Supplier_1 Unit Price 0.19000 -> 0.11000
- R_GATE1, R_GATE2, R_GATE3, R_GATE4, R_GATE5, R_GATE6: Mfr YAGEO -> Vishay Dale; Mfr P/N PA0402FRL570R01L -> RCS040210R0FKED; Supplier_1 P/N 13-PA0402FRL570R01LTR-ND -> 541-2879-2-ND; Supplier_1 Unit Price 0.31000 -> 0.11000
Connections:
- net GND: now also C_PACK_FLT1.1, C24.1; no longer C_PACK_FLT1.2
- net at C_CP1.2, R_MID1.2, U11.43 (VMID): now also C24.2
- net at R_PACK_FLT1.1, U11.38 (PACKP): now also C_PACK_FLT1.2; no longer C_PACK_FLT1.1
Other:
- note added: "Footprint wrong Replace"
- note added: "Wrong bulk cap"

Commit message: Updating stuff
Parts:
- added R17: 10k, Resistor_SMD:R_0603_1608Metric, symbol Device:R
- added R18, R19, R20, R21: R, symbol Device:R
- Q1: footprint Package_TO_SOT_SMD:SOT-223-3_TabPin2 -> _BMS:SOT230P700X185-4N
- R_CELL_FLT1, R_CELL_FLT2, R_CELL_FLT3, R_CELL_FLT4, R_CELL_FLT5, R_CELL_FLT6, R_CELL_FLT7: value 1000 Ω -> 1k; footprint Resistor_SMD:R_0402_1005Metric -> Resistor_SMD:R_0603_1608Metric; Mfr Vishay Dale -> YAGEO; Mfr P/N TNPW04021K00BEED -> AC0603FR-071KL; Supplier_1 P/N TNP1.00KDATR-ND -> 311-1KLDTR-ND; Supplier_1 Price @ QTY 1 -> (none); Supplier_1 Price @ Qty (none) -> 1; Supplier_1 Unit Price 0.23000 -> 0.10000; Supplier_2 (none) -> JLCPCB; Supplier_2 P/N (none) -> C116692; Supplier_2 Price @ Qty (none) -> 1; Supplier_2 Unit Price (none) -> 0.0025
- R_SRN_FLT1: value 100 Ω -> 100; footprint Resistor_SMD:R_0402_1005Metric -> Resistor_SMD:R_0603_1608Metric; Mfr Vishay Dale -> YAGEO; Mfr P/N RCS0402100RFKED -> RT0603BRD07100RL; Supplier_1 DigiKey -> Digikey; Supplier_1 P/N 541-2886-2-ND -> YAG1497TR-ND; Supplier_1 Price @ QTY 0.11000 -> (none); Supplier_1 Price @ Qty (none) -> 1; Supplier_1 Unit Price 1 -> 0.14000; Supplier_2 (none) -> JLCPCB; Supplier_2 P/N (none) -> C122970; Supplier_2 Price @ Qty (none) -> 1; Supplier_2 Unit Price (none) -> 0.0214
- R_SRP_FLT1: value 100 Ω -> 100; footprint Resistor_SMD:R_0402_1005Metric -> Resistor_SMD:R_0603_1608Metric; Mfr P/N RCS0402100RFKED -> CRCW0603100RFKEAHP; Supplier_1 DigiKey -> Digikey; Supplier_1 P/N 541-2886-2-ND -> 541-100STR-ND; Supplier_1 Price @ QTY 0.11000 -> (none); Supplier_1 Price @ Qty (none) -> 1; Supplier_1 Unit Price 1 -> 0.14000; Supplier_2 (none) -> JLCPCB; Supplier_2 P/N (none) -> C844725; Supplier_2 Price @ Qty (none) -> 1; Supplier_2 Unit Price (none) -> 0.0444
Connections:
- net C1: now also R_CELL_FLT6.2; no longer R_CELL_FLT6.1
- net C2: now also R_CELL_FLT5.2; no longer R_CELL_FLT5.1
- net C3: now also R_CELL_FLT4.2; no longer R_CELL_FLT4.1
- net C4: now also R_CELL_FLT3.2; no longer R_CELL_FLT3.1
- net C5: now also R_CELL_FLT2.2; no longer R_CELL_FLT2.1
- net CELL_0: now also R_CELL_FLT7.1; no longer R_CELL_FLT7.2
- net CELL_1: now also R_CELL_FLT6.1; no longer R_CELL_FLT6.2
- net CELL_2: now also R_CELL_FLT5.1; no longer R_CELL_FLT5.2
- net CELL_3: now also R_CELL_FLT4.1; no longer R_CELL_FLT4.2
- net CELL_4: now also R_CELL_FLT3.1; no longer R_CELL_FLT3.2
- net CELL_5: now also R_CELL_FLT2.1; no longer R_CELL_FLT2.2
- net CELL_6: now also R_CELL_FLT1.1; no longer R_CELL_FLT1.2
- net GND: now also R_CELL_FLT7.2, R18.1, R19.1, R20.1, R21.1; no longer R_CELL_FLT7.1
- net NTC1: now also R18.2
- net NTC2: now also R19.2
- net NTC3: now also R20.2
- net NTC4: now also R21.2
- net PACK-: now also R_SRN_FLT1.1; no longer R_SRN_FLT1.2
- net SRN: now also R_SRN_FLT1.2; no longer R_SRN_FLT1.1
- net TOP: now also R_CELL_FLT1.2; no longer R_CELL_FLT1.1
- net NSHDN renamed nSHDN
- net nSHDN: now also R17.1
- new net +3V3: R17.2

Commit message: Placement
Parts:
- removed C24, C_SRN_SRP1: 100 nF, Capacitor_SMD:C_0402_1005Metric, symbol Device:C
- removed R14, R16: 10k, Resistor_SMD:R_0402_1005Metric, symbol Device:R
- removed R17: 10k, Resistor_SMD:R_0603_1608Metric, symbol Device:R
- added C_MID1, C_SRP_SRN1: 100 nF, Capacitor_SMD:C_0603_1608Metric, symbol Device:C
- added C_PACK_E2, C_PACK_E3: ~, Capacitor_SMD:C_1206_3216Metric, symbol Device:C
- added R20, R21: 10k, Resistor_SMD:R_0603_1608Metric, symbol Device:R
- C19, C20, C21, C22, C23, C_CELL_FLT1, C_CELL_FLT2, C_CELL_FLT3, C_CELL_FLT4, C_CELL_FLT5, C_CELL_FLT6, C_PACK_FLT1: footprint Capacitor_SMD:C_0402_1005Metric -> Capacitor_SMD:C_0603_1608Metric; Mfr YAGEO -> Murata Electronics; Mfr P/N AC0402JRX7R9BB103 -> GRT1885C1E103FA02D; Supplier_1 P/N 13-AC0402JRX7R9BB103TR-ND -> 490-GRT1885C1E103FA02DTR-ND; Supplier_1 Unit Price 0.10000 -> 0.21000; Supplier_2 (none) -> JLCPCB; Supplier_2 P/N (none) -> C3836718; Supplier_2 Price @ Qty (none) -> 1; Supplier_2 Unit Price (none) -> 0.0482
- C_CP1: footprint Capacitor_SMD:C_0402_1005Metric -> Capacitor_SMD:C_0603_1608Metric
- C_PACK_E1: value 47 μF -> ~; Mfr KEMET -> (none); Mfr P/N A785KN476M1JLAS045 -> (none); Supplier_1 P/N 399-A785KN476M1JLAS045TR-ND -> (none); Supplier_1 Price @ QTY 0.97 -> (none)
- C_SRN_GND1, C_SRP_GND1: footprint Capacitor_SMD:C_0402_1005Metric -> Capacitor_SMD:C_0603_1608Metric; Mfr Murata Electronics -> YAGEO; Mfr P/N GRM155C71H104JE19D -> CC0603JRX7R9BB104; Supplier_1 P/N 490-GRM155C71H104JE19DTR-ND -> 311-1779-2-ND; Supplier_2 (none) -> JLCPCB; Supplier_2 P/N (none) -> C91183; Supplier_2 Price @ QTY (none) -> 1; Supplier_2 Unit Price (none) -> 0.0042
- Q2, Q3: value PSMN020-100YS -> PSMN3R7-100BSE; footprint _BMS:LFPAK56_1 -> _BMS:TO-263-2; Mfr P/N PSMN020-100YS,115 -> PSMN3R7-100BSEJ; Supplier_1 P/N 1727-4286-2-ND -> 1727-PSMN3R7-100BSEJTR-ND; Supplier_1 Unit Price 2.09000 -> 6.51
- R14: renamed from R13; footprint Resistor_SMD:R_0402_1005Metric -> Resistor_SMD:R_0603_1608Metric; Mfr Vishay Dale -> YAGEO; Mfr P/N TNPW040210K0BEED -> RC0603FR-0710KL; Supplier_1 P/N TNP10.0KDATR-ND -> 311-10.0KHRTR-ND; Supplier_1 Unit Price 0.23000 -> 0.10000; Supplier_2 (none) -> JLCPCB; Supplier_2 P/N (none) -> C98220; Supplier_2 Price @ Qty (none) -> 1; Supplier_2 Unit Price (none) -> 0.0013
- R15: footprint Resistor_SMD:R_0402_1005Metric -> Resistor_SMD:R_0603_1608Metric; Mfr Vishay Dale -> YAGEO; Mfr P/N TNPW040210K0BEED -> RC0603FR-0710KL; Supplier_1 P/N TNP10.0KDATR-ND -> 311-10.0KHRTR-ND; Supplier_1 Unit Price 0.23000 -> 0.10000; Supplier_2 (none) -> JLCPCB; Supplier_2 P/N (none) -> C98220; Supplier_2 Price @ Qty (none) -> 1; Supplier_2 Unit Price (none) -> 0.0013
- R16: renamed from R18; value R -> 10k; footprint (none) -> Resistor_SMD:R_0603_1608Metric
- R17: renamed from R19; value R -> 10k; footprint (none) -> Resistor_SMD:R_0603_1608Metric
- R18: renamed from R20; value R -> 10k; footprint (none) -> Resistor_SMD:R_0603_1608Metric
- R19: renamed from R21; value R -> 10k; footprint (none) -> Resistor_SMD:R_0603_1608Metric
- R_CHG_DRIVER1, R_CHG_MG1, R_CHG_MG2, R_DSG_DRIVER1, R_DSG_MG1, R_DSG_MG2: value 100 Ω -> 100; footprint Resistor_SMD:R_0402_1005Metric -> Resistor_SMD:R_0603_1608Metric; Mfr P/N RCS0402100RFKED -> CRCW0603100RFKEAHP; Supplier_1 DigiKey -> Digikey; Supplier_1 P/N 541-2886-2-ND -> 541-100STR-ND; Supplier_1 Price @ QTY 0.11000 -> (none); Supplier_1 Price @ Qty (none) -> 1; Supplier_1 Unit Price 1 -> 0.14000; Supplier_2 (none) -> JLCPCB; Supplier_2 P/N (none) -> C844725; Supplier_2 Price @ Qty (none) -> 1; Supplier_2 Unit Price (none) -> 0.0444
- R_GATE1, R_GATE2, R_GATE3, R_GATE4, R_GATE5, R_GATE6: footprint Resistor_SMD:R_0402_1005Metric -> Resistor_SMD:R_0603_1608Metric; Mfr P/N RCS040210R0FKED -> CRCW060310R0FKEAHP; Supplier_1 P/N 541-2879-2-ND -> 541-10.0STR-ND; Supplier_1 Unit Price 0.11000 -> 0.14000; Supplier_2 (none) -> JLCPCB; Supplier_2 P/N (none) -> C313648; Supplier_2 Price @ QTY (none) -> 1; Supplier_2 Unit Price (none) -> 0.0386
- R_MID1, R_PACK_FLT1: value 100 Ω -> 100; Mfr P/N RCA0603100RFKEAHP -> CRCW0603100RFKEAHP; Supplier_1 DigiKey -> Digikey; Supplier_1 P/N 541-3244-2-ND -> 541-100STR-ND; Supplier_1 Price @ QTY 1 -> (none); Supplier_1 Price @ Qty (none) -> 1; Supplier_1 Unit Price 0.10000 -> 0.14000; Supplier_2 (none) -> JLCPCB; Supplier_2 P/N (none) -> C844725; Supplier_2 Price @ Qty (none) -> 1; Supplier_2 Unit Price (none) -> 0.0444
- R_SRN_FLT1: Mfr YAGEO -> Vishay Dale; Mfr P/N RT0603BRD07100RL -> CRCW0603100RFKEAHP; Supplier_1 P/N YAG1497TR-ND -> 541-100STR-ND; Supplier_2 P/N C122970 -> C844725; Supplier_2 Unit Price 0.0214 -> 0.0444
- renumbered TP7 to TP10, TP1 to TP4, TP2 to TP5, TP3 to TP6, TP4 to TP7, TP5 to TP8, TP6 to TP9
Connections:
- net DRAIN: now also R_MID1.2; no longer R_MID1.1
- net DSG: now also R_DSG_DRIVER1.2; no longer R_DSG_DRIVER1.1
- net GND: now also C21.2, C22.2, C23.2, C_PACK_FLT1.2, C_SRN_GND1.1, C_SRP_GND1.2, C_MID1.2; no longer C21.1, C22.1, C23.1, C_PACK_FLT1.1, C_SRN_GND1.2, C_SRP_GND1.1
- net NTC1: now also C23.1, R21.1; no longer C23.2
- net NTC2: now also C22.1, R20.1; no longer C22.2, R15.1
- net NTC3: now also C21.1, R15.1; no longer C21.2
- net PACK+: now also C_PACK_E2.1, C_PACK_E3.1
- net PACK-: now also R_SRN_FLT1.2, C_PACK_E2.2, C_PACK_E3.2; no longer R_SRN_FLT1.1
- net SRN: now also C_SRN_GND1.2, R_SRN_FLT1.1, C_SRP_SRN1.1; no longer C_SRN_GND1.1, R_SRN_FLT1.2
- net SRP: now also C_SRP_GND1.1, C_SRP_SRN1.2; no longer C_SRP_GND1.2
- net at C19.2, R14.2, R15.2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: now also R20.2, R21.2
- net at Q4.2 (G): now also R_DSG_MG2.2; no longer R_DSG_MG2.1
- net at R_PACK_FLT1.1, U11.38 (PACKP): now also C_PACK_FLT1.1; no longer C_PACK_FLT1.2
- net at C_CP1.2, U11.43 (VMID): now also R_MID1.1, C_MID1.1; no longer R_MID1.2
- net at D_CHG_VGS1.1 (K), R_CHG_DRIVER1.2, R_CHG_MG2.1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: now also R_CHG_MG1.2; no longer R_CHG_MG1.1
- net at Q5.2 (G): now also R_DSG_MG1.1; no longer R_DSG_MG1.2
- net at Q2.2 (G): now also R_CHG_MG1.1; no longer R_CHG_MG1.2
- new net: D_CHG_VGS2.1 (K), R_DSG_DRIVER1.1, R_DSG_MG1.2, R_DSG_MG2.1, R_DSG_PUP1.1
Other:
- moved on the sheet: C_PACK_E1, D11

Commit message: Doing placement
Parts:
- added D13, D14: LED, LED_SMD:LED_0603_1608Metric, symbol Device:LED
- added R23, R24: R, Resistor_SMD:R_0603_1608Metric, symbol Device:R
- added TP12, TP13: TestPoint, TestPoint:TestPoint_Pad_D2.0mm, symbol Connector:TestPoint
Connections:
- net GND: now also D13.1 (K), D14.1 (K)
- net PACK+: now also R24.1, TP13.1
- net TOP: now also R23.1, TP12.1
- new net: D13.2 (A), R23.2
- new net: D14.2 (A), R24.2
Other:
- moved on the sheet: C19, C20, C21, C22, C23, C_3V3_1, C_CELL_FLT1, C_CELL_FLT2, C_CELL_FLT3, C_CELL_FLT4, C_CELL_FLT5, C_CELL_FLT6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

Commit message: Prelim placement done
Parts:
- removed TP12, TP13: TestPoint, TestPoint:TestPoint_Pad_D2.0mm, symbol Connector:TestPoint
- R_CHG_PUP1, R_DSG_PUP1: footprint Resistor_SMD:R_0402_1005Metric -> Resistor_SMD:R_0603_1608Metric
- U10, U5, U6, U7, U8, U9: footprint _BMS:SC70-6 -> _BMS:SC_4EEH-T1_GE3_VIS
Other:
- moved on the sheet: D13, D14, R23, R24

Commit message: Did a lot of routing
Connections:
- net TOP: no longer R_CHG_PUP1.2
- net at D_CHG_VGS1.1 (K), R_CHG_DRIVER1.2, R_CHG_MG1.2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: no longer R_CHG_PUP1.1
Other:
- moved on the sheet: R_CHG_PUP1
Changed lines of the file:
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@@
 		(lib_id "Device:R")
 		(at 245.11 245.11 0)
+		(mirror y)
 		(unit 1)
 		(exclude_from_sim no)
@@
 		(dnp no)
 		(property "Reference" "R_SRN_FLT1"
-			(at 251.968 243.84 0)
+			(at 238.252 243.84 0)
 			(effects
 				(font
@@
 		)
 		(property "Value" "100"
-			(at 251.968 246.38 0)
+			(at 238.252 246.38 0)
 			(effects
 				(font
@@
 		)
 		(property "Footprint" "Resistor_SMD:R_0603_1608Metric"
-			(at 243.332 245.11 90)
+			(at 246.888 245.11 90)
 			(effects
 				(font
@@
 	(symbol
 		(lib_id "Device:R")
-		(at 213.36 41.91 180)
+		(at 356.87 -287.02 180)
 		(unit 1)
 		(exclude_from_sim no)
@@
 		(dnp no)
 		(property "Reference" "R_CHG_PUP1"
-			(at 208.788 40.132 90)
+			(at 352.298 -288.798 90)
 			(effects
 				(font
@@
 		)
 		(property "Value" "10 MΩ"
-			(at 210.82 40.894 90)
+			(at 354.33 -288.036 90)
 			(effects
 				(font
@@
 		)
 		(property "Footprint" "Resistor_SMD:R_0603_1608Metric"
-			(at 215.138 41.91 90)
+			(at 358.648 -287.02 90)
 			(effects
 				(font
@@
 		)
 		(property "Datasheet" "https://www.koaspeer.com/pdfs/RK73H.pdf"
-			(at 213.36 41.91 0)
+			(at 356.87 -287.02 0)
 			(effects
 				(font
@@
 		)
 		(property "Description" "RES 10M OHM 1% 1/10W 0402"
-			(at 213.36 41.91 0)
+			(at 356.87 -287.02 0)
 			(effects
 				(font
@@
 		)
 		(property "Mfr" "KOA Speer Electronics, Inc."
-			(at 213.36 41.91 0)
+			(at 356.87 -287.02 0)
 			(effects
 				(font
@@
 		)
 		(property "Mfr P/N" "RK73H1ETTP1005F"
-			(at 213.36 41.91 0)
+			(at 356.87 -287.02 0)
 			(effects
 				(font
@@
 		)
 		(property "Supplier_1" "Digikey"
-			(at 213.36 41.91 90)
+			(at 356.87 -287.02 90)
 			(effects
 				(font
@@
 		)
 		(property "Supplier_1 P/N" "2019-RK73H1ETTP1005FTR-ND"
-			(at 213.36 41.91 90)
+			(at 356.87 -287.02 90)
 			(effects
 				(font
@@
 		)
 		(property "Supplier_1 Price @ QTY" "1"
-			(at 213.36 41.91 90)
+			(at 356.87 -287.02 90)
 			(effects
 				(font
@@
 		)
 		(property "Supplier_1 Unit Price" "0.10000"
-			(at 213.36 41.91 90)
+			(at 356.87 -287.02 90)
 			(effects
 				(font
@@
 		)
 		(property "Supplier_2" ""
-			(at 213.36 41.91 90)
+			(at 356.87 -287.02 90)
 			(effects
 				(font
@@
 		)
 		(property "Supplier_2 P/N" ""
-			(at 213.36 41.91 90)
+			(at 356.87 -287.02 90)
 			(effects
 				(font
@@
 		)
 		(property "Supplier_2 Price @ QTY" ""
-			(at 213.36 41.91 90)
+			(at 356.87 -287.02 90)
 			(effects
 				(font
@@
 		)
 		(property "Supplier_2 Unit Price" ""
-			(at 213.36 41.91 90)
+			(at 356.87 -287.02 90)
 			(effects
 				(font
@@
 		)
 		(property "Supplier_1 Price @ Qty" ""
-			(at 213.36 41.91 0)
+			(at 356.87 -287.02 0)
 			(effects
 				(font
@@
 		)
 		(property "Supplier_2 Price @ Qty" ""
-			(at 213.36 41.91 0)
+			(at 356.87 -287.02 0)
 			(effects
 				(font
