File: main.kicad_sch (KiCad schematic)
At the start: 0 parts

Commit message: Rev3 fixes
Other:
- added sheet CAN (can.kicad_sch)
- sheet external_io ports: added {CAN_LINE}; removed {I2C}
- sheet microcontroller ports: added {CAN}; removed BUS1{I2C}
