File: can.kicad_sch (KiCad schematic)
At the start: 13 parts, among them U19 MCP25625-E/ML, Y1 16MHz 12pF

Commit message: Adding in JST XH
Parts:
- removed R96: 10K, Resistor_SMD:R_0603_1608Metric, symbol Device:R_US
Connections:
- net CAN_STBY is gone; now on net GND: U19.15 (STBY)
Changed lines of the file:
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@@
 	(wire
 		(pts
-			(xy 110.49 105.41) (xy 129.54 105.41)
-		)
-		(stroke
-			(width 0)
-			(type default)
-		)
-	)
-	(wire
-		(pts
 			(xy 149.86 66.04) (xy 149.86 67.31)
 		)
@@
 	(wire
 		(pts
-			(xy 101.6 105.41) (xy 102.87 105.41)
-		)
-		(stroke
-			(width 0)
-			(type default)
-		)
-	)
-	(wire
-		(pts
 			(xy 168.91 105.41) (xy 186.69 105.41)
 		)
@@
 	(wire
 		(pts
+			(xy 101.6 105.41) (xy 129.54 105.41)
+		)
+		(stroke
+			(width 0)
+			(type default)
+		)
+	)
+	(wire
+		(pts
 			(xy 200.66 93.98) (xy 200.66 95.25)
 		)
@@
 					(unit 1)
 				)
-			)
-		)
-	)
-	(symbol
-		(lib_id "Device:R_US")
-		(at 106.68 105.41 270)
-		(unit 1)
-		(exclude_from_sim no)
-		(in_bom yes)
-		(on_board yes)
-		(dnp no)
-		(property "Reference" "R96"
-			(at 106.68 108.712 90)
-			(effects
-				(font
-					(size 1.27 1.27)
-				)
-			)
-		)
-		(property "Value" "10K"
-			(at 106.68 111.252 90)
-			(effects
-				(font
-					(size 1.27 1.27)
-				)
-			)
-		)
-		(property "Footprint" "Resistor_SMD:R_0603_1608Metric"
-			(at 106.426 106.426 90)
-			(effects
-				(font
-					(size 1.27 1.27)
-				)
-				(hide yes)
-			)
-		)
-		(property "Datasheet" "https://www.lcsc.com/product-detail/C4037161.html"
-			(at 106.68 105.41 0)
-			(effects
-				(font
-					(size 1.27 1.27)
-				)
-				(hide yes)
-			)
-		)
-		(property "Description" "10kΩ 100mW Thin Film Resistor ±50ppm/℃ ±1% 0603"
-			(at 106.68 105.41 0)
-			(effects
-				(font
-					(size 1.27 1.27)
-				)
-				(hide yes)
-			)
-		)
-		(property "LCSC Part" "C4037161"
-			(at 2.54 -2.54 0)
-			(effects
-				(font
-					(size 1.27 1.27)
-				)
-				(hide yes)
-			)
-		)
-		(property "Mfr" "Venkel"
-			(at 106.68 105.41 0)
-			(effects
-				(font
-					(size 1.27 1.27)
-				)
-				(hide yes)
-			)
-		)
-		(property "Mfr P/N" "TFCR0603-10W-C-1002FT"
-			(at 106.68 105.41 0)
-			(effects
-				(font
-					(size 1.27 1.27)
-				)
-				(hide yes)
-			)
-		)
-		(property "Supplier_1" "LCSC"
-			(at 106.68 105.41 0)
-			(effects
-				(font
-					(size 1.27 1.27)
-				)
-				(hide yes)
-			)
-		)
-		(property "Supplier_1 P/N" "C4037161"
-			(at 106.68 105.41 0)
-			(effects
-				(font
-					(size 1.27 1.27)
-				)
-				(hide yes)
-			)
-		)
-		(property "Supplier_1 Unit Price" ""
-			(at 106.68 105.41 0)
-			(effects
-				(font
-					(size 1.27 1.27)
-				)
-				(hide yes)
-			)
-		)
-		(property "Supplier_1 Price @ Qty" "1"
-			(at 106.68 105.41 0)
-			(effects
-				(font
-					(size 1.27 1.27)
-				)
-				(hide yes)
-			)
-		)
-		(property "Supplier_2" ""
-			(at 106.68 105.41 0)
-			(effects
-				(font
-					(size 1.27 1.27)
-				)
-				(hide yes)
-			)
-		)
-		(property "Supplier_2 P/N" ""
-			(at 106.68 105.41 0)
-			(effects
-				(font
-					(size 1.27 1.27)
-				)
-				(hide yes)
-			)
-		)
-		(property "Supplier_2 Unit Price" ""
-			(at 106.68 105.41 0)
-			(effects
-				(font
-					(size 1.27 1.27)
-				)
-				(hide yes)
-			)
-		)
-		(property "Supplier_2 Price @ Qty" ""
-			(at 106.68 105.41 0)
-			(effects
-				(font
-					(size 1.27 1.27)
-				)
-				(hide yes)
-			)
-		)
-		(property "JLCPCB Status" "JLC in-stock package match"
-			(at 106.68 105.41 0)
-			(effects
-				(font
-					(size 1.27 1.27)
-				)
-				(hide yes)
-			)
-		)
-		(property "Manufacturer_Name" ""
-			(at 106.68 105.41 90)
-			(effects
-				(font
-					(size 1.27 1.27)
-				)
-				(hide yes)
-			)
-		)
-		(property "Manufacturer_Part_Number" ""
-			(at 106.68 105.41 90)
-			(effects
-				(font
-					(size 1.27 1.27)
-				)
-				(hide yes)
-			)
-		)
-		(property "Mouser Part Number" ""
-			(at 106.68 105.41 90)
-			(effects
-				(font
-					(size 1.27 1.27)
-				)
-				(hide yes)
-			)
-		)
-		(property "Mouser Price/Stock" ""
-			(at 106.68 105.41 90)
-			(effects
-				(font
-					(size 1.27 1.27)
-				)
-				(hide yes)
-			)
-		)
-		(pin "1"
-		)
-		(pin "2"
-		)
-		(instances
-			(project "BMS"
-				(path "/124184ba-5d68-4d9f-8da6-acc6720ab30b/93f9b420-7cce-46a9-9201-666f07a18f85/5b507d3a-b1db-4604-a2a5-2db369d84636"
-					(reference "R96")
-					(unit 1)
-				)

Commit message: Adding JST XH and moving test points
Parts:
- added C25, C26: 100 nF, Capacitor_SMD:C_0603_1608Metric, symbol Device:C
- added R10: 10K, Resistor_SMD:R_0603_1608Metric, symbol Device:R_US
Connections:
- net +3V3: now also C25.1
- net +5V: now also C26.1
- net GND: now also C25.2, C26.2, R10.2; no longer U19.15 (STBY)
- new net CAN_STBY: R10.1, U19.15 (STBY)

Commit message: Finalizing BOM
Parts:
- C25: renamed from C104; JLCPCB Status JLC in-stock package match -> (none); Supplier_1 LCSC -> (none); Supplier_1 P/N C1647 -> (none); Supplier_2 (none) -> JLCPCB; Supplier_2 P/N (none) -> C1647
- C26: renamed from C105; JLCPCB Status JLC in-stock package match -> (none); LCSC Part C1647 -> (none); Supplier_1 LCSC -> (none); Supplier_1 P/N C1647 -> (none); Supplier_1 Price @ Qty 1 -> (none); Supplier_2 (none) -> JLCPCB; Supplier_2 P/N (none) -> C1647
- C29: renamed from C106; JLCPCB Status JLC in-stock package match -> (none); Supplier_1 LCSC -> (none); Supplier_1 P/N C1671 -> (none); Supplier_2 (none) -> JLCPCB; Supplier_2 P/N (none) -> C1671
- C30: renamed from C107; JLCPCB Status JLC in-stock package match -> (none); Supplier_1 LCSC -> (none); Supplier_1 P/N C1671 -> (none); Supplier_2 (none) -> JLCPCB; Supplier_2 P/N (none) -> C1671
- D22: renamed from D27; Supplier_1 JLCPCB -> (none); Supplier_1 P/N C315918 -> (none); Supplier_2 (none) -> JLCPCB; Supplier_2 P/N (none) -> C315918
- D23: renamed from D28; Supplier_1 JLCPCB -> (none); Supplier_1 P/N C315918 -> (none); Supplier_2 (none) -> JLCPCB; Supplier_2 P/N (none) -> C315918
- R48: renamed from R94; JLCPCB Status JLC in-stock package match -> (none); Supplier_1 P/N C4037161 -> (none); Supplier_2 (none) -> JLCPCB; Supplier_2 P/N (none) -> C4037161
- R49: renamed from R95; Supplier_1 LCSC -> (none); Supplier_1 P/N C4037161 -> (none); Supplier_2 (none) -> JLCPCB; Supplier_2 P/N (none) -> C4037161
- R50: renamed from R10; JLCPCB Status JLC in-stock package match -> (none); Supplier_1 LCSC -> (none); Supplier_1 P/N C4037161 -> (none); Supplier_2 (none) -> JLCPCB; Supplier_2 P/N (none) -> C4037161
- R51: renamed from R97; JLCPCB Status JLC in-stock package match -> (none); Supplier_1 LCSC -> (none); Supplier_1 P/N C22787 -> (none); Supplier_2 (none) -> JLCPCB; Supplier_2 P/N (none) -> C22787
- U11: renamed from U19; JLCPCB Status JLC in-stock package match -> (none); Supplier_1 LCSC -> (none); Supplier_1 P/N C481365 -> (none); Supplier_2 (none) -> JLCPCB; Supplier_2 P/N (none) -> C481365
- Y1: JLCPCB Status JLC in-stock package match -> (none); Supplier_1 LCSC -> (none); Supplier_1 P/N C426965 -> (none); Supplier_2 (none) -> JLCPCB; Supplier_2 P/N (none) -> C426965
- renumbered C26 to C27, C25 to C28
