File: cells.kicad_sch (KiCad schematic)
At the start: 2 parts, among them J13 Conn_01x07_Pin, J8 Conn_01x02_Pin

Commit message: Finalizing BOM
Parts:
- renumbered J13 to J8, J8 to J9
Changed lines of the file:
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@@
 		(on_board yes)
 		(dnp no)
-		(property "Reference" "J13"
+		(property "Reference" "J8"
 			(at 116.84 83.8201 0)
 			(effects
@@
 			(project ""
 				(path "/124184ba-5d68-4d9f-8da6-acc6720ab30b/93f9b420-7cce-46a9-9201-666f07a18f85/72bfe5e0-3464-488b-90f8-8143600a08cb"
-					(reference "J13")
+					(reference "J8")
 					(unit 1)
 				)
@@
 		(on_board yes)
 		(dnp no)
-		(property "Reference" "J8"
+		(property "Reference" "J9"
 			(at 118.11 109.2201 0)
 			(effects
@@
 			(project ""
 				(path "/124184ba-5d68-4d9f-8da6-acc6720ab30b/93f9b420-7cce-46a9-9201-666f07a18f85/72bfe5e0-3464-488b-90f8-8143600a08cb"
-					(reference "J8")
+					(reference "J9")
 					(unit 1)
 				)
