File: ntc.kicad_sch (KiCad schematic)
At the start: 3 parts, among them J10 Conn_01x02_Pin, J11 Conn_01x02_Pin, J9 Conn_01x02_Pin

Commit message: Finalizing BOM
Parts:
- renumbered J9 to J10, J10 to J11, J11 to J12
Changed lines of the file:
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@@
 		(dnp no)
 		(fields_autoplaced yes)
-		(property "Reference" "J10"
+		(property "Reference" "J11"
 			(at 148.59 91.4399 0)
 			(effects
@@
 			(project "BMS"
 				(path "/124184ba-5d68-4d9f-8da6-acc6720ab30b/93f9b420-7cce-46a9-9201-666f07a18f85/b732a1a5-50cf-4d70-be91-0bf27828f771"
-					(reference "J10")
+					(reference "J11")
 					(unit 1)
 				)
@@
 		(dnp no)
 		(fields_autoplaced yes)
-		(property "Reference" "J9"
+		(property "Reference" "J10"
 			(at 148.59 81.2799 0)
 			(effects
@@
 			(project "BMS"
 				(path "/124184ba-5d68-4d9f-8da6-acc6720ab30b/93f9b420-7cce-46a9-9201-666f07a18f85/b732a1a5-50cf-4d70-be91-0bf27828f771"
-					(reference "J9")
+					(reference "J10")
 					(unit 1)
 				)
@@
 		(dnp no)
 		(fields_autoplaced yes)
-		(property "Reference" "J11"
+		(property "Reference" "J12"
 			(at 148.59 101.5999 0)
 			(effects
@@
 			(project "BMS"
 				(path "/124184ba-5d68-4d9f-8da6-acc6720ab30b/93f9b420-7cce-46a9-9201-666f07a18f85/b732a1a5-50cf-4d70-be91-0bf27828f771"
-					(reference "J11")
+					(reference "J12")
 					(unit 1)
 				)
@@
 		(dnp no)
 		(fields_autoplaced yes)
-		(property "Reference" "#PWR093"
+		(property "Reference" "#PWR089"
 			(at 135.89 93.98 0)
 			(effects
@@
 			(project "BMS"
 				(path "/124184ba-5d68-4d9f-8da6-acc6720ab30b/93f9b420-7cce-46a9-9201-666f07a18f85/b732a1a5-50cf-4d70-be91-0bf27828f771"
-					(reference "#PWR093")
+					(reference "#PWR089")
 					(unit 1)
 				)
@@
 		(dnp no)
 		(fields_autoplaced yes)
-		(property "Reference" "#PWR094"
+		(property "Reference" "#PWR090"
 			(at 135.89 104.14 0)
 			(effects
@@
 			(project "BMS"
 				(path "/124184ba-5d68-4d9f-8da6-acc6720ab30b/93f9b420-7cce-46a9-9201-666f07a18f85/b732a1a5-50cf-4d70-be91-0bf27828f771"
-					(reference "#PWR094")
+					(reference "#PWR090")
 					(unit 1)
 				)
@@
 		(dnp no)
 		(fields_autoplaced yes)
-		(property "Reference" "#PWR092"
+		(property "Reference" "#PWR088"
 			(at 135.89 83.82 0)
 			(effects
@@
 			(project ""
 				(path "/124184ba-5d68-4d9f-8da6-acc6720ab30b/93f9b420-7cce-46a9-9201-666f07a18f85/b732a1a5-50cf-4d70-be91-0bf27828f771"
-					(reference "#PWR092")
+					(reference "#PWR088")
 					(unit 1)
 				)
